File: V0/V0.0/schematics/smart penetrometer/_autosave-smart penetrometer.kicad_pcb (KiCad board)
At the start: 2 copper layers, 33 x 74.9 mm, 20 parts, among them J1 XLR3_Switched, J2 Conn_01x11_Female, U1 4001, U2 DS3231M, U3 Battery_Input, U4 4023, U5 ADS1115IDGS, U6 3v3_Voltage_Regulator, U7 Solar_Input

Commit message: malichi update
Parts:
- moved U7 2.54 mm to (115.6, 80.0)
Routing:
- net VCC: track 33.5 -> 37.9 mm
- net GND: track 41.1 -> 43.6 mm
- net Net-(BT1-Pad1): track 36.8 -> 35.0 mm
Changed lines of the file:
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@@
     (thickness 1.6)
     (drawings 4)
-    (tracks 218)
+    (tracks 220)
     (zones 0)
     (modules 20)
@@
   )
   (module kitest:Battery_Input (layer F.Cu)
-    (at 115.57 82.55)
+    (at 115.57 80.01)
     (fp_text reference U7 (at 0 1.27) (layer F.SilkS)
       (effects (font (size 1 1) (thickness 0.15)))
@@
   (segment (start 126.09999 129.17001) (end 126.09999 113.17502) (width 0.25) (layer B.Cu) (net 4))
   (segment (start 118.11 137.16) (end 126.09999 129.17001) (width 0.25) (layer B.Cu) (net 4))
-  (segment (start 110.83999 84.74001) (end 111.76 83.82) (width 0.25) (layer F.Cu) (net 5))
   (segment (start 110.83999 91.74999) (end 110.83999 84.74001) (width 0.25) (layer F.Cu) (net 5))
   (segment (start 111.165 92.075) (end 110.83999 91.74999) (width 0.25) (layer F.Cu) (net 5))
@@
   (segment (start 127 116.43) (end 129.13 114.3) (width 0.25) (layer B.Cu) (net 5))
   (segment (start 127 121.92) (end 127 116.43) (width 0.25) (layer B.Cu) (net 5))
+  (segment (start 110.83999 82.20001) (end 111.76 81.28) (width 0.25) (layer F.Cu) (net 5))
+  (segment (start 110.83999 84.74001) (end 110.83999 82.20001) (width 0.25) (layer F.Cu) (net 5))
   (segment (start 110.85999 114.805008) (end 110.85999 127.36999) (width 0.25) (layer B.Cu) (net 6))
   (segment (start 117.569999 108.094999) (end 110.85999 114.805008) (width 0.25) (layer B.Cu) (net 6))
@@
   (segment (start 119.38 91.44) (end 119.38 91.44) (width 0.25) (layer B.Cu) (net 32))
   (via (at 119.38 91.44) (size 0.8) (drill 0.4) (layers F.Cu B.Cu) (net 32))
+  (via (at 114.3 80.065001) (size 0.8) (drill 0.4) (layers F.Cu B.Cu) (net 32))
+  (segment (start 119.38 90.874315) (end 119.38 91.44) (width 0.25) (layer F.Cu) (net 32))
   (segment (start 120.719315 89.535) (end 121.49 89.535) (width 0.25) (layer F.Cu) (net 32))
   (segment (start 119.38 90.874315) (end 120.719315 89.535) (width 0.25) (layer F.Cu) (net 32))
-  (segment (start 119.38 91.44) (end 119.38 90.874315) (width 0.25) (layer F.Cu) (net 32))
-  (segment (start 113.085001 82.769663) (end 113.085001 80.065001) (width 0.25) (layer F.Cu) (net 32))
-  (segment (start 120.150338 89.835) (end 113.085001 82.769663) (width 0.25) (layer F.Cu) (net 32))
+  (segment (start 120.150338 89.835) (end 114.3 83.984662) (width 0.25) (layer F.Cu) (net 32))
   (segment (start 121.19 89.835) (end 120.150338 89.835) (width 0.25) (layer F.Cu) (net 32))
+  (segment (start 114.3 83.984662) (end 114.3 80.065001) (width 0.25) (layer F.Cu) (net 32))
   (segment (start 121.49 89.535) (end 121.19 89.835) (width 0.25) (layer F.Cu) (net 32))
-  (segment (start 113.085001 80.065001) (end 113.085001 80.065001) (width 0.25) (layer F.Cu) (net 32))
-  (via (at 113.085001 80.065001) (size 0.8) (drill 0.4) (layers F.Cu B.Cu) (net 32))
-  (segment (start 114.879999 80.065001) (end 116.84 78.105) (width 0.25) (layer B.Cu) (net 32))
-  (segment (start 113.085001 80.065001) (end 114.879999 80.065001) (width 0.25) (layer B.Cu) (net 32))
+  (segment (start 116.260001 78.105) (end 114.3 80.065001) (width 0.25) (layer B.Cu) (net 32))
+  (segment (start 116.84 78.105) (end 116.260001 78.105) (width 0.25) (layer B.Cu) (net 32))
   (segment (start 111.35 91.85) (end 111.35 104.14) (width 0.25) (layer B.Cu) (net 33))
   (segment (start 116.84 86.36) (end 111.35 91.85) (width 0.25) (layer B.Cu) (net 33))
@@
   (segment (start 139.7 91.03) (end 139.7 83.82) (width 0.25) (layer F.Cu) (net 34))
   (segment (start 137.16 93.57) (end 139.7 91.03) (width 0.25) (layer F.Cu) (net 34))
-  (segment (start 120.02 83.82) (end 119.38 83.82) (width 0.25) (layer F.Cu) (net 34))
-  (segment (start 128.27 92.07) (end 120.02 83.82) (width 0.25) (layer F.Cu) (net 34))
   (segment (start 128.27 93.57) (end 128.27 92.07) (width 0.25) (layer F.Cu) (net 34))
+  (segment (start 119.38 83.18) (end 121.605 85.405) (width 0.25) (layer F.Cu) (net 34))
+  (segment (start 119.38 81.28) (end 119.38 83.18) (width 0.25) (layer F.Cu) (net 34))
+  (segment (start 121.605 85.405) (end 120.02 83.82) (width 0.25) (layer F.Cu) (net 34))
+  (segment (start 128.27 92.07) (end 121.605 85.405) (width 0.25) (layer F.Cu) (net 34))
   (segment (start 137.16 86.77) (end 128.27 86.77) (width 0.25) (layer F.Cu) (net 35))
   (segment (start 128.27 81.28) (end 125.73 78.74) (width 0.25) (layer F.Cu) (net 35))
