File: V0/V0.0/schematics/smart penetrometer/smart penetrometer.sch (KiCad schematic (older format))
At the start: 15 parts, among them J1 XLR3_Switched, J2 Conn_01x03_Female, J3 Conn_01x02_Female, J4 Conn_01x04_Female, U1 4001, U2 DS3231M, U3 Battery_Input, U4 4023, U5 ADS1115IDGS

Commit message: malichi updtae
Parts:
- added U?: BD33GA5WEFJ, Package_SO:HTSOP-8-1EP_3.9x4.9mm_P1.27mm_EP2.4x3.2mm, symbol Regulator_Linear:BD33GA5WEFJ
Connections:
- new net: U?.3 (GND), U?.4 (GND), U?.6 (GND), U?.7 (GND), U?.9 (GND)
Changed lines of the file:
@@
+	1    0    0    -1
+$EndComp
+$Comp
+L Regulator_Linear:BD33GA5WEFJ U?
+U 1 1 61FDF517
+P 2700 2050
+F 0 "U?" H 2700 2292 50  0000 C CNN
+F 1 "BD33GA5WEFJ" H 2700 2201 50  0000 C CNN
+F 2 "Package_SO:HTSOP-8-1EP_3.9x4.9mm_P1.27mm_EP2.4x3.2mm" H 2700 1950 50  0001 C CNN
+F 3 "http://rohmfs.rohm.com/en/products/databook/datasheet/ic/power/linear_regulator/bdxxga5wefj-e.pdf" H 2700 1950 50  0001 C CNN
+	1    2700 2050
 	1    0    0    -1
 $EndComp

Commit message: malichi update
Parts:
- removed J2: Conn_01x03_Female, Connector_PinSocket_2.54mm:PinSocket_1x03_P2.54mm_Horizontal, symbol Connector:Conn_01x03_Female
- removed J3: Conn_01x02_Female, Connector_PinSocket_2.54mm:PinSocket_1x02_P2.54mm_Horizontal, symbol Connector:Conn_01x02_Female
- removed J4: Conn_01x04_Female, Connector_PinSocket_2.54mm:PinSocket_1x04_P2.54mm_Horizontal, symbol Connector:Conn_01x04_Female
- removed U?: BD33GA5WEFJ, Package_SO:HTSOP-8-1EP_3.9x4.9mm_P1.27mm_EP2.4x3.2mm, symbol Regulator_Linear:BD33GA5WEFJ
- added C1: C_0.1uF, Capacitor_SMD:C_1206_3216Metric, symbol Device:C_Small
- added C2: C_10uF, Capacitor_SMD:C_1206_3216Metric, symbol Device:C_Small
- added D1: D_Zener_Small, Diode_SMD:D_SMC, symbol Device:D_Zener_Small
- added D2: B320, Diode_SMD:D_SMC, symbol Diode:B320
- added D3: B350, Diode_SMD:D_SMC, symbol Diode:B350
- added J2: Conn_01x11_Female, Connector_PinSocket_2.54mm:PinSocket_1x11_P2.54mm_Horizontal, symbol Connector:Conn_01x11_Female
- added U6: 3v3_Voltage_Regulator, smart penetrometer footprints:BD433M2FP3_CE2, symbol smart-penetrometer-rescue:3v3_Voltage_Regulator
- added U7: Solar_Input, kitest:Battery_Input, symbol smart-penetrometer-rescue:Battery_Input-kitest-kitest-rescue
Connections:
- net VCC: now also D2.2 (A), D3.2 (A), U7.1 (Pos); no longer J1.2
- net at A1.1 (3V3), R5.1, R6.1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: now also A2.30 (VIN), C2.2, J2.10 (Pin_10), J2.6 (Pin_6), J2.7 (Pin_7), U6.3 (VOUT); no longer A2.17 (3V3)
- net at A2.19 (A0): now also J2.11 (Pin_11)
- net at A2.23 (A4), R5.2, U2.15 (SDA)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: now also J2.4 (Pin_4)
- net at A2.24 (A5), R6.2, U2.16 (SCL)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: now also J2.3 (Pin_3)
- net at J1.3: now also C1.1, D1.1 (K), U6.1 (VIN); no longer A2.30 (VIN)
- net at A2.5 (D2): now also J2.5 (Pin_5)
- net at U5.5 (AIN1): now also J2.1 (Pin_1)
- net at U5.4 (AIN0): now also J2.2 (Pin_2)
- new net: D2.1 (K), D3.1 (K), J1.2
- new net GNDREF: C1.2, C2.1, D1.2 (A), J2.8 (Pin_8), J2.9 (Pin_9), U6.2 (CTR), U6.4 (GND), U7.2 (Neg)
- no-connect marks 27 -> 30
Other:
- moved on the sheet: U3

Commit message: malichi update
Connections:
- net GND: now also C1.2, C2.1, D1.2 (A), U6.2 (CTR), U6.4 (GND), U7.2 (Neg)
- net GNDREF: no longer C1.2, C2.1, D1.2 (A), U6.2 (CTR), U6.4 (GND), U7.2 (Neg)
Changed lines of the file:
@@
 Wire Wire Line
 	2500 4350 2500 3100
-$Comp
-L power:GNDREF #PWR08
-U 1 1 61FF764F
-P 2650 2850
-F 0 "#PWR08" H 2650 2600 50  0001 C CNN
-F 1 "GNDREF" H 2655 2677 50  0000 C CNN
-F 2 "" H 2650 2850 50  0001 C CNN
-F 3 "" H 2650 2850 50  0001 C CNN
-	1    2650 2850
-	1    0    0    -1
-$EndComp
-$Comp
-L power:GNDREF #PWR02
-U 1 1 61FF8208
-P 2300 2500
-F 0 "#PWR02" H 2300 2250 50  0001 C CNN
-F 1 "GNDREF" V 2305 2372 50  0000 R CNN
-F 2 "" H 2300 2500 50  0001 C CNN
-F 3 "" H 2300 2500 50  0001 C CNN
-	1    2300 2500
-	0    1    1    0
-$EndComp
 Wire Wire Line
 	2800 2850 2800 3100
@@
 $EndComp
 $Comp
-L power:GNDREF #PWR010
-U 1 1 61FFB798
-P 3000 2850
-F 0 "#PWR010" H 3000 2600 50  0001 C CNN
-F 1 "GNDREF" V 3005 2722 50  0000 R CNN
-F 2 "" H 3000 2850 50  0001 C CNN
-F 3 "" H 3000 2850 50  0001 C CNN
-	1    3000 2850
-	0    -1   -1   0
-$EndComp
-$Comp
 L Device:C_Small C1
 U 1 1 61FFC277
@@
 Wire Wire Line
 	2500 3100 2500 2850
-$Comp
-L power:GNDREF #PWR05
-U 1 1 61FFCC13
-P 2300 2850
-F 0 "#PWR05" H 2300 2600 50  0001 C CNN
-F 1 "GNDREF" H 2305 2677 50  0000 C CNN
-F 2 "" H 2300 2850 50  0001 C CNN
-F 3 "" H 2300 2850 50  0001 C CNN
-	1    2300 2850
-	1    0    0    -1
-$EndComp
 Connection ~ 2800 2850
 Connection ~ 2500 2850
@@
 $EndComp
 $Comp
-L power:GNDREF #PWR07
-U 1 1 620037A9
-P 2300 3100
-F 0 "#PWR07" H 2300 2850 50  0001 C CNN
-F 1 "GNDREF" V 2305 2972 50  0000 R CNN
-F 2 "" H 2300 3100 50  0001 C CNN
-F 3 "" H 2300 3100 50  0001 C CNN
-	1    2300 3100
-	0    1    1    0
-$EndComp
-$Comp
 L Connector:Conn_01x11_Female J2
 U 1 1 62004E69
@@
 $EndComp
 $Comp
-L power:GNDREF #PWR013
-U 1 1 6205315E
-P 3250 2100
-F 0 "#PWR013" H 3250 1850 50  0001 C CNN
-F 1 "GNDREF" H 3255 1927 50  0000 C CNN
-F 2 "" H 3250 2100 50  0001 C CNN
-F 3 "" H 3250 2100 50  0001 C CNN
-	1    3250 2100
-	1    0    0    -1
-$EndComp
-$Comp
 L power:VCC #PWR014
 U 1 1 62053C3C
@@
 	4450 2400 4100 2400
 Connection ~ 4100 2400
+$Comp
+L power:GND #PWR?
+U 1 1 6206C9B7
+P 2300 2500
+F 0 "#PWR?" H 2300 2250 50  0001 C CNN
+F 1 "GND" V 2305 2372 50  0000 R CNN
+F 2 "" H 2300 2500 50  0001 C CNN
+F 3 "" H 2300 2500 50  0001 C CNN
+	1    2300 2500
+	0    1    1    0
+$EndComp
+$Comp
+L power:GND #PWR?
+U 1 1 6206F54E
+P 3250 2100
+F 0 "#PWR?" H 3250 1850 50  0001 C CNN
+F 1 "GND" H 3255 1927 50  0000 C CNN
+F 2 "" H 3250 2100 50  0001 C CNN
+F 3 "" H 3250 2100 50  0001 C CNN
+	1    3250 2100
+	1    0    0    -1
+$EndComp
+$Comp
+L power:GND #PWR?
+U 1 1 62071F32
+P 2300 3100
+F 0 "#PWR?" H 2300 2850 50  0001 C CNN
+F 1 "GND" H 2305 2927 50  0000 C CNN
+F 2 "" H 2300 3100 50  0001 C CNN
+F 3 "" H 2300 3100 50  0001 C CNN
+	1    2300 3100
+	1    0    0    -1
+$EndComp
+$Comp
+L power:GND #PWR?
+U 1 1 62074C30
+P 2300 2850
+F 0 "#PWR?" H 2300 2600 50  0001 C CNN
+F 1 "GND" H 2305 2677 50  0000 C CNN
+F 2 "" H 2300 2850 50  0001 C CNN
+F 3 "" H 2300 2850 50  0001 C CNN
+	1    2300 2850
+	1    0    0    -1
+$EndComp
+$Comp
+L power:GND #PWR?
+U 1 1 620772C4
+P 2650 2850
+F 0 "#PWR?" H 2650 2600 50  0001 C CNN
+F 1 "GND" H 2655 2677 50  0000 C CNN
+F 2 "" H 2650 2850 50  0001 C CNN
+F 3 "" H 2650 2850 50  0001 C CNN
+	1    2650 2850
+	1    0    0    -1
+$EndComp
+$Comp
+L power:GND #PWR?
+U 1 1 62079E29
+P 3000 2850
+F 0 "#PWR?" H 3000 2600 50  0001 C CNN
+F 1 "GND" H 3005 2677 50  0000 C CNN
+F 2 "" H 3000 2850 50  0001 C CNN
+F 3 "" H 3000 2850 50  0001 C CNN
+	1    3000 2850
+	1    0    0    -1
+$EndComp
 $EndSCHEMATC
