File: V0/V0.0/schematics/smart penetrometer/smart penetrometer.kicad_pcb (KiCad board)
At the start: 2 copper layers, 33 x 74.9 mm, 20 parts, among them J1 XLR3_Switched, J2 Conn_01x11_Female, U1 4001, U2 DS3231M, U3 Battery_Input, U4 4023, U5 ADS1115IDGS, U6 3v3_Voltage_Regulator, U7 Solar_Input

Commit message: malichi update
Parts:
- moved U3 2.54 mm to (135.9, 80.0)
- moved U7 2.54 mm to (115.6, 80.0)
- moved J2 1.27 mm to (113.0, 148.6)
Routing:
- net GNDS: track 20.1 -> 60.3 mm, vias 0 -> 1
- net GND: track 41.1 -> 73.1 mm, vias 0 -> 3
- net Net-(A2-Pad5): track 50.8 -> 39.2 mm, vias 0 -> 2
- net Net-(A2-Pad24): track 113.3 -> 105.1 mm
- net VCC: track 33.5 -> 40.4 mm
- net Net-(A2-Pad23): track 105.6 -> 107.8 mm
- net Net-(BT1-Pad1): track 36.8 -> 35.0 mm
- net Net-(A1-Pad1): track 148.0 -> 146.4 mm, vias 1 -> 2
- net Net-(A2-Pad19): track 17.3 -> 18.6 mm
- net Net-(J2-Pad1): track 3.88 -> 5.15 mm
- net Net-(J2-Pad2): track 6.47 -> 7.15 mm
Other:
- board text added: "+"
- board text added: "-"
- board text added: "02/08/2022"
- board text added: "3V3 VOLTAGE REGULATOR"
- board text added: "A0"
- board text added: "ACCELEROMETER"
- board text added: "ARDUINO NANO"
- board text added: "BME 280"
- board text added: "CS"
- board text added: "GEOPHONE"
- board text added: "GND"
- board text added: "INT2"
- board text added: "Malichi Flemming II"
- board text added: "SCHOTTKY DIODES"
- board text added: "SCL"
- board text added: "SDA"
- board text added: "SMART PENETROMETER V5"
- board text added: "TDS"
- board text added: "VCC"
- board text added: "ZENER DIODE"
