File: hardware_design/V1.0/V1.0/PCB/smart penetrometer V1.0/smart penetrometer V1.0.sch (KiCad schematic (older format))
At the start: 24 parts, among them J1 XLR3_Switched, J2 Conn_01x11_Female, U2 DS3231M, U3 Battery_Input, U4 4023, U5 ADS1115IDGS, U6 3v3_Voltage_Regulator, U7 Solar_Input

Commit message: update
Parts:
- added U?: 23k256SRAM, symbol smart-penetrometer-V1.0-rescue:23k256SRAM
Connections:
- net at A2.12 (D9): now also A1.2 (CS)
- net at A2.13 (D10): now also U?.1 (CS); no longer A1.2 (CS)
- net at A1.3 (MOSI), A2.14 (D11): now also U?.5 (SI)
- net at A1.5 (MISO), A2.15 (D12): now also U?.2 (SO)
- net at A1.4 (CLK), A2.16 (D13): now also U?.6 (SCK)
- net at A2.17 (3V3): now also A1.1 (3V3), C2.2, J2.10 (Pin_10), J2.6 (Pin_6), J2.7 (Pin_7), R5.1, R6.1, U2.2 (VCC), U4.13, U5.8 (VDD), U6.3 (VOUT), U?.4 (Vss)
- net at C1.1, D1.1 (K), J1.3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: now also A2.30 (VIN)
Changed lines of the file:
@@
 Wire Wire Line
 	4800 2900 4800 4750
-Wire Wire Line
-	4650 4550 4850 4550
 $Comp
 L power:GND #PWR04
@@
 NoConn ~ 4850 4250
 NoConn ~ 4850 4350
-NoConn ~ 4850 4450
 $Comp
 L smart-penetrometer-V1.0-rescue:Battery_Input-kitest-kitest-rescue-smart-penetrometer-rescue U3
@@
 NoConn ~ 5550 3150
 Wire Wire Line
-	4650 2600 4650 4550
-Wire Wire Line
 	3500 3100 3500 5800
 Wire Wire Line
@@
 $EndComp
 Wire Wire Line
-	3950 4350 2500 4350
-Wire Wire Line
 	2500 4350 2500 3100
 Wire Wire Line
@@
 	2800 3100 3500 3100
 Connection ~ 3500 3100
-Wire Wire Line
-	3500 3100 5250 3100
 $Comp
 L Device:C_Small C2
@@
 Wire Wire Line
 	4100 2400 3600 2400
-NoConn ~ 5450 3150
 $Comp
 L power:VCC #PWR0101
@@
 	0    1    1    0
 $EndComp
-Wire Wire Line
-	5250 3150 5250 3100
-Connection ~ 5250 3100
-Wire Wire Line
-	5250 3100 6050 3100
 $Comp
 L Diode:B320 D2
@@
 	2050 1350 2050 1150
 Connection ~ 2050 1150
+Wire Wire Line
+	5450 3150 5450 3100
+Connection ~ 5450 3100
+Wire Wire Line
+	5450 3100 6050 3100
+Wire Wire Line
+	3500 3100 5450 3100
+Wire Wire Line
+	5250 3150 4300 3150
+Wire Wire Line
+	4300 3150 4300 4350
+Wire Wire Line
+	2500 4350 3950 4350
+Connection ~ 3950 4350
+Wire Wire Line
+	3950 4350 4300 4350
+$Comp
+L smart-penetrometer-V1.0-rescue:23k256SRAM U?
+U 1 1 62BD39C8
+P 2850 5150
+F 0 "U?" H 2850 5665 50  0000 C CNN
+F 1 "23k256SRAM" H 2850 5574 50  0000 C CNN
+F 2 "" H 2850 5150 50  0001 C CNN
+F 3 "" H 2850 5150 50  0001 C CNN
+	1    2850 5150
+	1    0    0    -1
+$EndComp
+Wire Wire Line
+	4850 4450 4650 4450
+Wire Wire Line
+	4650 2600 4650 4450
+Wire Wire Line
+	2500 4550 2500 4900
+Wire Wire Line
+	2500 4550 4850 4550
+Wire Wire Line
+	4700 4650 3400 4650
+Wire Wire Line
+	3400 4650 3400 5400
+Wire Wire Line
+	3400 5400 3200 5400
+Connection ~ 4700 4650
+Wire Wire Line
+	4800 4750 2450 4750
+Wire Wire Line
+	2450 4750 2450 5050
+Wire Wire Line
+	2450 5050 2500 5050
+Connection ~ 4800 4750
+Wire Wire Line
+	4750 4850 3600 4850
+Wire Wire Line
+	3600 4850 3600 5250
+Wire Wire Line
+	3600 5250 3200 5250
+Connection ~ 4750 4850
+Wire Wire Line
+	2500 5400 2500 5800
+Wire Wire Line
+	2500 5800 3500 5800
+Connection ~ 3500 5800
+NoConn ~ 3200 5050
+NoConn ~ 2500 5250
 $EndSCHEMATC
