File: V1/V1.0.0/hardware_design/PCB/smart penetrometer update/_autosave-smart penetrometer update.sch (KiCad schematic (older format))
At the start: 44 parts, among them J1 XLR3_Switched, J2 Conn_01x11_Female, J3 Conn_01x02_Female, U1 LM22676MR-5, U10 FS8205A, U11 DW01, U2 DS3231M, U3 Battery_Input, U4 4023, U5 ADS1115IDGS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

Commit message: Fix PCB Design
Several traces missing in PCB Design.
Parts:
- A1: symbol smart-penetrometer-update-rescue:SD_Card_Module-Charleslabs_Parts-kitest-rescue-smart-penetrometer-rescue-smart-penetro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 -> smart~penetrometer~update-rescue:SD_Card_Module-Charleslabs_Parts-kitest-rescue-smart-penetrometer-rescue-smart-penetro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
- A2: symbol smart-penetrometer-update-rescue:Arduino_Nano_v3.x-MCU_Module-kitest-rescue-smart-penetrometer-rescue-smart-penetromete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 -> smart~penetrometer~update-rescue:Arduino_Nano_v3.x-MCU_Module-kitest-rescue-smart-penetrometer-rescue-smart-penetromete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
- C12: symbol smart-penetrometer-update-rescue:CP1_Small-Device -> smart~penetrometer~update-rescue:CP1_Small-Device
- J1: symbol Connector:XLR3_Switched -> smart~penetrometer~update-rescue:XLR3_Switched-Connector
- J2: symbol Connector:Conn_01x11_Female -> smart~penetrometer~update-rescue:Conn_01x11_Female-Connector
- J3: symbol Connector:Conn_01x02_Female -> smart~penetrometer~update-rescue:Conn_01x02_Female-Connector
- U10: symbol smart-penetrometer-update-rescue:FS8205A-smart-penetrometer-rescue-smart-penetrometer-update-rescue -> smart~penetrometer~update-rescue:FS8205A-smart-penetrometer-rescue-smart-penetrometer-update-rescue
- U11: symbol smart-penetrometer-update-rescue:DW01-smart-penetrometer-rescue-smart-penetrometer-update-rescue -> smart~penetrometer~update-rescue:DW01-smart-penetrometer-rescue-smart-penetrometer-update-rescue
- U3, U7: symbol smart-penetrometer-update-rescue:Battery_Input-kitest-kitest-rescue-smart-penetrometer-rescue-smart-penetrometer-update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 -> smart~penetrometer~update-rescue:Battery_Input-kitest-kitest-rescue-smart-penetrometer-rescue-smart-penetrometer-update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
- U6: symbol smart-penetrometer-update-rescue:3v3_Voltage_Regulator-smart-penetrometer-rescue-smart-penetrometer-update-rescue -> smart~penetrometer~update-rescue:3v3_Voltage_Regulator-smart-penetrometer-rescue-smart-penetrometer-update-rescue
- U9: symbol smart-penetrometer-update-rescue:SRAM(23K256)-smart-penetrometer-update-rescue -> smart~penetrometer~update-rescue:SRAM(23K256)-smart-penetrometer-update-rescue
Changed lines of the file:
@@
 EESchema Schematic File Version 5
-EELAYER 36 0
+EELAYER 43 0
 EELAYER END
 $Descr A4 11693 8268
@@
 $EndComp
 $Comp
-L smart-penetrometer-update-rescue:CP1_Small-Device C12
+L smart~penetrometer~update-rescue:CP1_Small-Device C12
 U 1 1 62819F8F
 P 4200 1000
@@
 $EndComp
 $Comp
-L Connector:Conn_01x02_Female J3
+L smart~penetrometer~update-rescue:Conn_01x02_Female-Connector J3
 U 1 1 63030D60
 P 850 5850
@@
 $EndComp
 $Comp
-L smart-penetrometer-update-rescue:Battery_Input-kitest-kitest-rescue-smart-penetrometer-rescue-smart-penetrometer-update-rescue U7
+L smart~penetrometer~update-rescue:Battery_Input-kitest-kitest-rescue-smart-penetrometer-rescue-smart-penetrometer-update-rescue-smart-penetrometer-update-rescue U7
 U 1 1 62051BA4
 P 3400 1950
@@
 $EndComp
 $Comp
-L smart-penetrometer-update-rescue:Battery_Input-kitest-kitest-rescue-smart-penetrometer-rescue-smart-penetrometer-update-rescue U3
+L smart~penetrometer~update-rescue:Battery_Input-kitest-kitest-rescue-smart-penetrometer-rescue-smart-penetrometer-update-rescue-smart-penetrometer-update-rescue U3
 U 1 1 60A6877D
 P 4200 750
@@
 $EndComp
 $Comp
-L smart-penetrometer-update-rescue:DW01-smart-penetrometer-rescue-smart-penetrometer-update-rescue U11
+L smart~penetrometer~update-rescue:DW01-smart-penetrometer-rescue-smart-penetrometer-update-rescue U11
 U 1 1 62805E03
 P 4300 1450
@@
 $EndComp
 $Comp
-L Connector:Conn_01x11_Female J2
+L smart~penetrometer~update-rescue:Conn_01x11_Female-Connector J2
 U 1 1 62004E69
 P 7000 6200
@@
 $EndComp
 $Comp
-L smart-penetrometer-update-rescue:3v3_Voltage_Regulator-smart-penetrometer-rescue-smart-penetrometer-update-rescue U6
+L smart~penetrometer~update-rescue:3v3_Voltage_Regulator-smart-penetrometer-rescue-smart-penetrometer-update-rescue U6
 U 1 1 61FF42DE
 P 3100 2600
@@
 $EndComp
 $Comp
-L Connector:XLR3_Switched J1
+L smart~penetrometer~update-rescue:XLR3_Switched-Connector J1
 U 1 1 60DFB15F
 P 3950 4050
@@
 $EndComp
 $Comp
-L smart-penetrometer-update-rescue:SRAM(23K256)-smart-penetrometer-update-rescue U9
+L smart~penetrometer~update-rescue:SRAM(23K256)-smart-penetrometer-update-rescue U9
 U 1 1 62EB656F
 P 2500 6900
@@
 $EndComp
 $Comp
-L smart-penetrometer-update-rescue:SD_Card_Module-Charleslabs_Parts-kitest-rescue-smart-penetrometer-rescue-smart-penetrometer-update-rescue A1
+L smart~penetrometer~update-rescue:SD_Card_Module-Charleslabs_Parts-kitest-rescue-smart-penetrometer-rescue-smart-penetrometer-update-rescue A1
 U 1 1 60A4A816
 P 5350 2750
@@
 $EndComp
 $Comp
-L smart-penetrometer-update-rescue:FS8205A-smart-penetrometer-rescue-smart-penetrometer-update-rescue U10
+L smart~penetrometer~update-rescue:FS8205A-smart-penetrometer-rescue-smart-penetrometer-update-rescue U10
 U 1 1 62819888
 P 2600 1250
@@
 $EndComp
 $Comp
-L smart-penetrometer-update-rescue:Arduino_Nano_v3.x-MCU_Module-kitest-rescue-smart-penetrometer-rescue-smart-penetrometer-update-rescue A2
+L smart~penetrometer~update-rescue:Arduino_Nano_v3.x-MCU_Module-kitest-rescue-smart-penetrometer-rescue-smart-penetrometer-update-rescue A2
 U 1 1 60A40C30
 P 5350 4150
