File: V1/V1.0.0/hardware_design/PCB/smart penetrometer update/smart penetrometer update.kicad_pcb (KiCad board)
At the start: 2 copper layers, 33 x 74.9 mm, 25 parts, among them J1 XLR3_Switched, J2 Conn_01x11_Female, U1 4001, U2 DS3231M, U3 Battery_Input, U4 4023, U5 ADS1115IDGS, U6 3v3_Voltage_Regulator, U7 Solar_Input, U8 FS8205A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

Commit message: no change
Parts:
- added C10: C_0.1uF, Capacitor_SMD:C_1206_3216Metric, F.Cu at (127.0, 144.8)
- added C11: C_0.1uF, Capacitor_SMD:C_1206_3216Metric, B.Cu at (129.5, 133.3)
- added C3: C_10uF, Capacitor_SMD:C_1206_3216Metric, B.Cu at (137.2, 85.1)
- added C5: C_0.047uF, Capacitor_SMD:C_1206_3216Metric, B.Cu at (127.0, 90.2)
- added C6: C_0.47uF, Capacitor_SMD:C_1206_3216Metric, F.Cu at (113.2, 100.3)
- added C7: C_0.047uF, Capacitor_SMD:C_1206_3216Metric, F.Cu at (114.3, 110.5)
- added C8: C_10uF, Capacitor_SMD:C_1206_3216Metric, B.Cu at (127.0, 86.4)
- added C9: C_0.1uF, Capacitor_SMD:C_1206_3216Metric, B.Cu at (157.3, 41.9)
- added D4: PMEG6045ETP, Diode_SMD:D_SOD-128, F.Cu at (191.8, 58.4)
- added J3: Conn_01x02_Female, Connector_PinSocket_2.54mm:PinSocket_1x02_P2.54mm_Horizontal, F.Cu at (171.4, 78.7)
- added L1: L, Inductor_SMD:L_1206_3216Metric, F.Cu at (123.2, 102.9)
- added R1: R_1MOhm, Resistor_SMD:R_1206_3216Metric, B.Cu at (138.4, 113.0)
- added R2: R_1MOhm, Resistor_SMD:R_1206_3216Metric, F.Cu at (172.5, 55.9)
- added R3: R_800Ohm, Resistor_SMD:R_1206_3216Metric, F.Cu at (123.4, 108.0)
- added R4: R_800Ohm, Resistor_SMD:R_1206_3216Metric, F.Cu at (256.3, 45.7)
- added R7: R_Small_US, Resistor_SMD:R_1206_3216Metric, B.Cu at (133.3, 144.8)
- added R8: R_Small_US, Resistor_SMD:R_1206_3216Metric, B.Cu at (113.0, 143.5)
- added U1: LM22676MR-5, Package_SO:TI_SO-PowerPAD-8, B.Cu at (137.2, 91.4)
- added U8: ADS1120-PW, Package_SO:TSSOP-16_4.4x5mm_P0.65mm, F.Cu at (124.5, 132.1)
- added U9: SRAM(23K256), smart penetrometer footprints:23K256T-E&slash_SN, F.Cu at (124.5, 139.7)
- U10: renamed from U8; footprint smart penetrometer footprints:FS8205A -> smart penetrometer footprints:DUAL_MOSFET(FS8205A); moved to B.Cu
- U11: renamed from U9; footprint smart penetrometer footprints:DW01 -> smart penetrometer footprints:BATTERY_PROTECTION_IC(DW01A)
- moved U10 15.3 mm to (114.3, 119.4), turned to 90 degrees
- renumbered C3 to C12, R2 to R10, R1 to R9
Connections:
- net Net-(C3-Pad1) renamed -BATT
- net VCC renamed +BATT
- A2 pad 17: Net-(A1-Pad1) -> Net-(A2-Pad17)
- A2 pad 30: Net-(A2-Pad30) -> Net-(A1-Pad1)
- J1 pad 3: Net-(C1-Pad1) -> Net-(C3-Pad2)
- R9 pad 1: Net-(R1-Pad1) -> Net-(R9-Pad1)
Routing:
- net Net-(U10-Pad5): track 15.1 -> 0.00 mm
- net Net-(R9-Pad1): track 0.00 -> 15.1 mm
- net Net-(U8-Pad4): track 0.00 -> 7.84 mm
- net Net-(U10-Pad4): track 7.84 -> 0.00 mm
- net Net-(U8-Pad1): track 0.00 -> 5.40 mm
- net Net-(U10-Pad1): track 5.40 -> 0.00 mm

Commit message: Fix PCB Design
Several traces missing in PCB Design.
Routing:
- net GNDREF: track 2.54 -> 10.5 mm, vias 0 -> 1
Other:
- net class Default removed
