File: V0/V0.4.1/hardware_design/PCB/smart penetrometer/smart penetrometer.kicad_pcb (KiCad board)
At the start: 4 copper layers, 29 x 83.8 mm, 22 parts, among them J1 Conn_01x02_Female, J2 XLR3_Switched, J3 Conn_01x07_Female, U1 ADS1120-PW, U2 DS3231M, U3 4023, U4 ADS1115IDGS

Commit message: PCB V0.4.1 UPDATE
Parts:
- added G***: LOGO, kitest:uofsc_logo_0_75in, B.Cu at (181.5, 76.9)
- added J4: Screw_Terminal, TerminalBlock:TerminalBlock_bornier-2_P5.08mm, B.Cu at (171.3, 65.7)
- added R7: R_1.9kOhm, Resistor_SMD:R_1206_3216Metric, B.Cu at (186.0, 62.9)
- added U5: VO615A, footprints:Vishay_VOS615A, B.Cu at (179.2, 63.6)
- moved BT1 1.06 mm to (180.6, 69.6)
Connections:
- A1 pad 11: unconnected-(A1-Pad11) -> 5V0
- A1 pad 27: unconnected-(A1-Pad27) -> 5V0
Routing:
- net 5V0: track 0.00 -> 97.9 mm
- net Net-(J4-Pad2): track 0.00 -> 11.0 mm
- net Net-(J4-Pad1): track 0.00 -> 5.44 mm
- net Net-(R7-Pad1): track 0.00 -> 2.19 mm
- net Net-(BT1-Pad1): track 33.3 -> 32.1 mm
Other:
- board text added: "BY MALICHI FLEMMING II 05/19/2023"
- board text added: "GEO"
- board text added: "GND"
- board text added: "OFF"
- board text added: "ON"
- board text added: "SPECIES V0.4.1"
- board text added: "TDS"
- board text added: "THERMO"

Commit message: PCB UPDATE
Parts:
- added G***: LOGO, kitest:ARTS_lab_logo, B.Cu at (180.5, 86.9)
- moved G*** 1.00 mm to (180.5, 76.7)
Routing:
- added copper zone on In2.Cu, net 3V3
- added copper zone on In1.Cu, net GND
- removed copper zone on In1.Cu, net 3V3
- removed copper zone on In2.Cu, net GND
Other:
- board text added: "OPTOCOUPLER"
- board text added: "TERMINALS"
