File: V0/V0.4.1/hardware_design/PCB/smart penetrometer/smart penetrometer.kicad_sch (KiCad schematic)
At the start: 22 parts, among them J1 Conn_01x02_Female, J2 XLR3_Switched, J3 Conn_01x07_Female, U1 ADS1120-PW, U2 DS3231M, U3 4023, U4 ADS1115IDGS

Commit message: PCB V0.4.1 UPDATE
Parts:
- added J4: Screw_Terminal, TerminalBlock:TerminalBlock_bornier-2_P5.08mm, symbol Connector:Screw_Terminal_01x02
- added R7: R_1.9kOhm, Resistor_SMD:R_1206_3216Metric, symbol Device:R_Small_US
- added U5: VO615A, footprints:Vishay_VOS615A, symbol Isolator:VO615A
Connections:
- net GND: now also R7.2
- net 5V0: now reaches A1.11 (D8)
- net 5V0: now also A1.27 (+5V), U5.4
- new net: R7.1, U5.3
- new net: J4.1 (Pin_1), U5.1
- new net: J4.2 (Pin_2), U5.2
- no-connect marks 31 -> 29
Other:
- note added: "OPTOCOUPLER"

Commit message: update
Parts:
- U1: value ADS1120-PW -> ADS1120IRVAR
- U4: value ADS1115IDGS -> ADS1115IRUGT
Other:
- note added: "GEOPHONE ADC W/ AMPLIFIER"
- note removed: "GEOPHONE AMPLIFIER"
- moved on the sheet: U4
Changed lines of the file:
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@@
   (junction (at 139.7 45.72) (diameter 0) (color 0 0 0 0)
   )
-  (no_connect (at 257.81 142.24))
-  (no_connect (at 237.49 149.86))
+  (no_connect (at 231.14 142.24))
+  (no_connect (at 251.46 149.86))
   (no_connect (at 55.88 138.43))
   (no_connect (at 91.44 151.13))
-  (no_connect (at 257.81 152.4))
+  (no_connect (at 231.14 152.4))
   (no_connect (at 143.51 111.76))
   (no_connect (at 88.9 53.34))
   (no_connect (at 55.88 153.67))
   (no_connect (at 168.91 99.06))
-  (no_connect (at 237.49 152.4))
+  (no_connect (at 251.46 152.4))
   (no_connect (at 168.91 129.54))
   (no_connect (at 143.51 106.68))
@@
     (effects (font (size 1.27 1.27)) (justify left bottom))
   )
-  (text "GEOPHONE AMPLIFIER" (at 224.79 130.81 0)
+  (text "GEOPHONE ADC W/ AMPLIFIER" (at 224.79 130.81 0)
     (effects (font (size 1.27 1.27)) (justify left bottom))
   )
@@
     (effects (font (size 1.27 1.27)) (justify left bottom))
   )
-  (global_label "SDA" (shape bidirectional) (at 257.81 149.86 0) (fields_autoplaced)
-    (effects (font (size 1.27 1.27)) (justify left))
-    (property "Intersheet References" "${INTERSHEET_REFS}" (id 0) (at 263.7912 149.9394 0)
-      (effects (font (size 1.27 1.27)) (justify left) hide)
+  (global_label "SDA" (shape bidirectional) (at 231.14 149.86 180) (fields_autoplaced)
+    (effects (font (size 1.27 1.27)) (justify right))
+    (property "Intersheet References" "${INTERSHEET_REFS}" (id 0) (at 225.1588 149.9394 0)
+      (effects (font (size 1.27 1.27)) (justify right) hide)
     )
   )
@@
     )
   )
-  (global_label "GEO_AMP_0" (shape input) (at 237.49 144.78 180) (fields_autoplaced)
-    (effects (font (size 1.27 1.27)) (justify right))
-    (property "Intersheet References" "${INTERSHEET_REFS}" (id 0) (at 224.3726 144.7006 0)
-      (effects (font (size 1.27 1.27)) (justify right) hide)
+  (global_label "GEO_AMP_0" (shape input) (at 251.46 144.78 0) (fields_autoplaced)
+    (effects (font (size 1.27 1.27)) (justify left))
+    (property "Intersheet References" "${INTERSHEET_REFS}" (id 0) (at 264.5774 144.7006 0)
+      (effects (font (size 1.27 1.27)) (justify left) hide)
     )
   )
@@
     )
   )
-  (global_label "SCL" (shape input) (at 257.81 147.32 0) (fields_autoplaced)
-    (effects (font (size 1.27 1.27)) (justify left))
-    (property "Intersheet References" "${INTERSHEET_REFS}" (id 0) (at 263.7307 147.2406 0)
-      (effects (font (size 1.27 1.27)) (justify left) hide)
-    )
-  )
-  (global_label "GEO_AMP_1" (shape input) (at 237.49 147.32 180) (fields_autoplaced)
-    (effects (font (size 1.27 1.27)) (justify right))
-    (property "Intersheet References" "${INTERSHEET_REFS}" (id 0) (at 224.3726 147.2406 0)
-      (effects (font (size 1.27 1.27)) (justify right) hide)
+  (global_label "SCL" (shape input) (at 231.14 147.32 180) (fields_autoplaced)
+    (effects (font (size 1.27 1.27)) (justify right))
+    (property "Intersheet References" "${INTERSHEET_REFS}" (id 0) (at 225.2193 147.2406 0)
+      (effects (font (size 1.27 1.27)) (justify right) hide)
+    )
+  )
+  (global_label "GEO_AMP_1" (shape input) (at 251.46 147.32 0) (fields_autoplaced)
+    (effects (font (size 1.27 1.27)) (justify left))
+    (property "Intersheet References" "${INTERSHEET_REFS}" (id 0) (at 264.5774 147.2406 0)
+      (effects (font (size 1.27 1.27)) (justify left) hide)
     )
   )
@@
     )
   )
-  (global_label "3V3" (shape input) (at 247.65 134.62 90) (fields_autoplaced)
-    (effects (font (size 1.27 1.27)) (justify left))
-    (property "Intersheet References" "${INTERSHEET_REFS}" (id 0) (at 247.5706 128.6993 90)
-      (effects (font (size 1.27 1.27)) (justify left) hide)
+  (global_label "3V3" (shape input) (at 241.3 134.62 0) (fields_autoplaced)
+    (effects (font (size 1.27 1.27)) (justify left))
+    (property "Intersheet References" "${INTERSHEET_REFS}" (id 0) (at 247.2207 134.6994 0)
+      (effects (font (size 1.27 1.27)) (justify right) hide)
     )
   )
@@
     (pin "2")
   )
-  (symbol (lib_id "Analog_ADC:ADS1115IDGS") (at 247.65 147.32 0) (unit 1)
-    (in_bom yes) (on_board yes)
-    (property "Reference" "U4" (id 0) (at 247.65 146.05 0))
-    (property "Value" "ADS1115IDGS" (id 1) (at 234.95 134.62 0))
-    (property "Footprint" "kitest:10X2QFN" (id 2) (at 247.65 160.02 0)
-      (effects (font (size 1.27 1.27)) hide)
-    )
-    (property "Datasheet" "http://www.ti.com/lit/ds/symlink/ads1113.pdf" (id 3) (at 246.38 170.18 0)
+  (symbol (lib_id "Analog_ADC:ADS1115IDGS") (at 241.3 147.32 0) (mirror y) (unit 1)
+    (in_bom yes) (on_board yes)
+    (property "Reference" "U4" (id 0) (at 241.3 146.05 0))
+    (property "Value" "ADS1115IRUGT" (id 1) (at 256.54 137.16 0))
+    (property "Footprint" "kitest:10X2QFN" (id 2) (at 241.3 160.02 0)
+      (effects (font (size 1.27 1.27)) hide)
+    )
+    (property "Datasheet" "http://www.ti.com/lit/ds/symlink/ads1113.pdf" (id 3) (at 242.57 170.18 0)
       (effects (font (size 1.27 1.27)) hide)
     )
@@
     (pin "2")
   )
-  (symbol (lib_id "power:GND") (at 247.65 157.48 0) (unit 1)
-    (in_bom yes) (on_board yes)
-    (property "Reference" "#PWR018" (id 0) (at 247.65 163.83 0)
-      (effects (font (size 1.27 1.27)) hide)
-    )
-    (property "Value" "GND" (id 1) (at 248.92 161.29 0))
-    (property "Footprint" "" (id 2) (at 247.65 157.48 0)
-      (effects (font (size 1.27 1.27)) hide)
-    )
-    (property "Datasheet" "" (id 3) (at 247.65 157.48 0)
+  (symbol (lib_id "power:GND") (at 241.3 157.48 0) (mirror y) (unit 1)
+    (in_bom yes) (on_board yes)
+    (property "Reference" "#PWR018" (id 0) (at 241.3 163.83 0)
+      (effects (font (size 1.27 1.27)) hide)
+    )
+    (property "Value" "GND" (id 1) (at 240.03 161.29 0))
+    (property "Footprint" "" (id 2) (at 241.3 157.48 0)
+      (effects (font (size 1.27 1.27)) hide)
+    )
+    (property "Datasheet" "" (id 3) (at 241.3 157.48 0)
       (effects (font (size 1.27 1.27)) hide)
     )
@@
     (in_bom yes) (on_board yes)
     (property "Reference" "U1" (id 0) (at 72.39 144.78 0))
-    (property "Value" "ADS1120-PW" (id 1) (at 72.39 147.32 0))
+    (property "Value" "ADS1120IRVAR" (id 1) (at 72.39 147.32 0))
     (property "Footprint" "Package_DFN_QFN:VQFN-16-1EP_3x3mm_P0.5mm_EP1.45x1.45mm_ThermalVias" (id 2) (at 80.01 132.08 0)
       (effects (font (size 1.27 1.27)) (justify left) hide)
@@
     )
     (path "/e3a1353f-e4bf-4da6-9946-0b37beaca1d8"
-      (reference "U1") (unit 1) (value "ADS1120-PW") (footprint "Package_DFN_QFN:VQFN-16-1EP_3x3mm_P0.5mm_EP1.45x1.45mm_ThermalVias")
+      (reference "U1") (unit 1) (value "ADS1120IRVAR") (footprint "Package_DFN_QFN:VQFN-16-1EP_3x3mm_P0.5mm_EP1.45x1.45mm_ThermalVias")
     )
     (path "/4beaa797-c457-4c8d-a454-ffc2fb829970"
@@
     )
     (path "/1377caaf-f76e-484b-aac7-0bb96ebdd4f7"
-      (reference "U4") (unit 1) (value "ADS1115IDGS") (footprint "kitest:10X2QFN")
+      (reference "U4") (unit 1) (value "ADS1115IRUGT") (footprint "kitest:10X2QFN")
     )
     (path "/3eb75b6b-3499-4125-a6dc-a33406dd9a5e"

Commit message: update
Parts:
- C6: value C_Small -> C_0.1uF
- R5, R6: value R_Small_US -> R_1kOhm
- U3: value 4023 -> BME260
