File: V0/V0.5/V0.5.0/hardware_design/PCB/smart penetrometer/smart penetrometer0.4.2.kicad_pcb (KiCad board)
At the start: 4 copper layers, 29 x 83.8 mm, 27 parts, among them J1 Conn_01x02_Female, J2 XLR3_Switched, J3 Conn_01x07_Female, J4 Screw_Terminal, U1 ADS1120-PW, U2 DS3231M, U3 4023, U4 ADS1115IDGS, U5 VO615A

Commit message: update
Parts:
- moved R5 18.9 mm to (189.4, 94.4), turned to 90 degrees
- moved R6 11.4 mm to (177.9, 95.5)
Routing:
- net SDA: track 77.7 -> 74.9 mm
- net SCL: track 78.7 -> 77.4 mm
Changed lines of the file:
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@@
   )
   (footprint "Resistor_SMD:R_1206_3216Metric" (layer "F.Cu")
-    (at 178.054 109.474)
+    (at 189.38 94.376 90)
     (descr "Resistor SMD 1206 (3216 Metric), square (rectangular) end terminal, IPC_7351 nominal, (Body size source: IPC-SM-782 page 72, https://www.pcb-3d.com/wordpress/wp-content/uploads/ipc-sm-782a_amendment_1_and_2.pdf), generated with kicad-footprint-generator")
     (tags "resistor")
@@
     (property "Sheetname" "")
     (attr smd)
-    (fp_text reference "R5" (at -4.064 0) (layer "F.SilkS")
+    (fp_text reference "R5" (at -4.064 0 90) (layer "F.SilkS")
         (effects (font (size 1 1) (thickness 0.15)))
     )
-    (fp_text value "R_Small_US" (at 0 1.82) (layer "F.Fab")
+    (fp_text value "R_Small_US" (at 0 1.82 90) (layer "F.Fab")
         (effects (font (size 1 1) (thickness 0.15)))
     )
-    (fp_text user "${REFERENCE}" (at 0 0) (layer "F.Fab")
+    (fp_text user "${REFERENCE}" (at 0 0 90) (layer "F.Fab")
         (effects (font (size 0.8 0.8) (thickness 0.12)))
     )
@@
     (fp_line (start 1.6 0.8) (end -1.6 0.8)
       (stroke (width 0.1) (type solid)) (layer "F.Fab"))
-    (pad "1" smd roundrect (at -1.4625 0) (size 1.125 1.75) (layers "F.Cu" "F.Paste" "F.Mask") (roundrect_rratio 0.222222)
+    (pad "1" smd roundrect (at -1.4625 0 90) (size 1.125 1.75) (layers "F.Cu" "F.Paste" "F.Mask") (roundrect_rratio 0.222222)
       (net 17 "3V3") (pintype "passive"))
-    (pad "2" smd roundrect (at 1.4625 0) (size 1.125 1.75) (layers "F.Cu" "F.Paste" "F.Mask") (roundrect_rratio 0.222222)
+    (pad "2" smd roundrect (at 1.4625 0 90) (size 1.125 1.75) (layers "F.Cu" "F.Paste" "F.Mask") (roundrect_rratio 0.222222)
       (net 23 "SDA") (pintype "passive"))
     (model "${KICAD6_3DMODEL_DIR}/Resistor_SMD.3dshapes/R_1206_3216Metric.wrl"
@@
   )
   (footprint "Resistor_SMD:R_1206_3216Metric" (layer "F.Cu")
-    (at 178.054 106.934)
+    (at 177.924 95.54)
     (descr "Resistor SMD 1206 (3216 Metric), square (rectangular) end terminal, IPC_7351 nominal, (Body size source: IPC-SM-782 page 72, https://www.pcb-3d.com/wordpress/wp-content/uploads/ipc-sm-782a_amendment_1_and_2.pdf), generated with kicad-footprint-generator")
     (tags "resistor")
@@
   (segment (start 179.066 118.4505) (end 178.566 118.4505) (width 0.25) (layer "F.Cu") (net 17))
   (via (at 176.53 104.14) (size 1) (drill 0.6) (layers "F.Cu" "B.Cu") (net 17))
-  (via (at 176.53 109.474) (size 1) (drill 0.6) (layers "F.Cu" "B.Cu") (net 17))
+  (via (at 189.38 95.9) (size 1) (drill 0.6) (layers "F.Cu" "B.Cu") (net 17))
   (via (at 175.26 138.684) (size 1) (drill 0.6) (layers "F.Cu" "B.Cu") (net 17))
-  (via (at 176.53 106.934) (size 1) (drill 0.6) (layers "F.Cu" "B.Cu") (net 17))
+  (via (at 176.4 95.54) (size 1) (drill 0.6) (layers "F.Cu" "B.Cu") (net 17))
   (via (at 179.07 117.348) (size 0.8) (drill 0.4) (layers "F.Cu" "B.Cu") (free) (net 17))
   (via (at 176.53 101.346) (size 1) (drill 0.6) (layers "F.Cu" "B.Cu") (net 17))
@@
   (segment (start 187.706 140.096) (end 185.39 142.412) (width 0.25) (layer "B.Cu") (net 19))
   (segment (start 184.285 78.605) (end 184.84 78.605) (width 0.25) (layer "F.Cu") (net 23))
+  (segment (start 186.428 90.162) (end 182.88 86.614) (width 0.25) (layer "F.Cu") (net 23))
+  (segment (start 186.97 90.704) (end 186.428 90.162) (width 0.25) (layer "F.Cu") (net 23))
+  (segment (start 186.97 107.03) (end 186.97 90.704) (width 0.25) (layer "F.Cu") (net 23))
   (segment (start 182.88 80.01) (end 184.285 78.605) (width 0.25) (layer "F.Cu") (net 23))
-  (segment (start 188.468 109.22) (end 188.468 132.588) (width 0.25) (layer "F.Cu") (net 23))
-  (segment (start 190.5 94.234) (end 182.88 86.614) (width 0.25) (layer "F.Cu") (net 23))
+  (segment (start 189.1795 92.9135) (end 189.38 92.9135) (width 0.25) (layer "F.Cu") (net 23))
+  (segment (start 186.97 90.704) (end 189.1795 92.9135) (width 0.25) (layer "F.Cu") (net 23))
+  (segment (start 184.685 109.315) (end 186.97 107.03) (width 0.25) (layer "F.Cu") (net 23))
   (segment (start 182.88 86.614) (end 182.88 80.01) (width 0.25) (layer "F.Cu") (net 23))
-  (segment (start 188.468 109.22) (end 190.5 107.188) (width 0.25) (layer "F.Cu") (net 23))
-  (segment (start 179.6755 109.315) (end 184.685 109.315) (width 0.25) (layer "F.Cu") (net 23))
-  (segment (start 188.468 132.588) (end 182.753 138.303) (width 0.25) (layer "F.Cu") (net 23))
-  (segment (start 190.5 107.188) (end 190.5 94.234) (width 0.25) (layer "F.Cu") (net 23))
-  (segment (start 179.5165 109.474) (end 179.6755 109.315) (width 0.25) (layer "F.Cu") (net 23))
+  (segment (start 186.938 111.568) (end 186.938 134.118) (width 0.25) (layer "F.Cu") (net 23))
+  (segment (start 186.938 134.118) (end 182.753 138.303) (width 0.25) (layer "F.Cu") (net 23))
+  (segment (start 184.685 109.315) (end 186.938 111.568) (width 0.25) (layer "F.Cu") (net 23))
+  (segment (start 189.38 92.9135) (end 189.221 92.7545) (width 0.25) (layer "F.Cu") (net 23))
   (segment (start 182.753 138.303) (end 181.344001 138.303) (width 0.25) (layer "F.Cu") (net 23))
   (segment (start 188.468 109.22) (end 184.78 109.22) (width 0.25) (layer "B.Cu") (net 23))
   (segment (start 184.78 109.22) (end 184.685 109.315) (width 0.25) (layer "B.Cu") (net 23))
-  (segment (start 179.5165 106.934) (end 179.6755 106.775) (width 0.25) (layer "F.Cu") (net 24))
+  (segment (start 181.454001 137.668) (end 182.019001 137.668) (width 0.25) (layer "F.Cu") (net 24))
+  (segment (start 183.17 108.29) (end 184.685 106.775) (width 0.25) (layer "F.Cu") (net 24))
+  (segment (start 179.3865 95.54) (end 179.5455 95.381) (width 0.25) (layer "F.Cu") (net 24))
   (segment (start 181.864 78.74) (end 181.864 86.868) (width 0.25) (layer "F.Cu") (net 24))
-  (segment (start 181.864 86.868) (end 189.738 94.742) (width 0.25) (layer "F.Cu") (net 24))
+  (segment (start 182.019001 137.668) (end 183.17 136.517) (width 0.25) (layer "F.Cu") (net 24))
   (segment (start 183.388 77.216) (end 181.864 78.74) (width 0.25) (layer "F.Cu") (net 24))
-  (segment (start 186.69 108.78) (end 186.69 132.997) (width 0.25) (layer "F.Cu") (net 24))
-  (segment (start 186.69 132.997) (end 182.019001 137.668) (width 0.25) (layer "F.Cu") (net 24))
-  (segment (start 189.738 105.41) (end 188.468 106.68) (width 0.25) (layer "F.Cu") (net 24))
+  (segment (start 186.2 91.204) (end 186.148 91.152) (width 0.25) (layer "F.Cu") (net 24))
+  (segment (start 179.5455 95.381) (end 186.199 95.381) (width 0.25) (layer "F.Cu") (net 24))
+  (segment (start 184.685 106.775) (end 186.2 105.26) (width 0.25) (layer "F.Cu") (net 24))
+  (segment (start 186.2 95.38) (end 186.2 91.204) (width 0.25) (layer "F.Cu") (net 24))
   (segment (start 184.721 77.216) (end 183.388 77.216) (width 0.25) (layer "F.Cu") (net 24))
-  (segment (start 189.738 94.742) (end 189.738 105.41) (width 0.25) (layer "F.Cu") (net 24))
-  (segment (start 184.685 106.775) (end 186.69 108.78) (width 0.25) (layer "F.Cu") (net 24))
+  (segment (start 186.199 95.381) (end 186.2 95.38) (width 0.25) (layer "F.Cu") (net 24))
   (segment (start 184.84 77.335) (end 184.721 77.216) (width 0.25) (layer "F.Cu") (net 24))
-  (segment (start 182.019001 137.668) (end 181.454001 137.668) (width 0.25) (layer "F.Cu") (net 24))
-  (segment (start 179.6755 106.775) (end 184.685 106.775) (width 0.25) (layer "F.Cu") (net 24))
+  (segment (start 181.864 86.868) (end 186.148 91.152) (width 0.25) (layer "F.Cu") (net 24))
+  (segment (start 186.2 105.26) (end 186.2 95.38) (width 0.25) (layer "F.Cu") (net 24))
+  (segment (start 183.17 136.517) (end 183.17 108.29) (width 0.25) (layer "F.Cu") (net 24))
   (segment (start 184.685 106.775) (end 188.373 106.775) (width 0.25) (layer "B.Cu") (net 24))
   (segment (start 188.373 106.775) (end 188.468 106.68) (width 0.25) (layer "B.Cu") (net 24))
