File: V0/V0.5/V0.5.0/hardware_design/PCB/smart penetrometer/smart penetrometer.kicad_sch (KiCad schematic)
At the start: 25 parts, among them J1 Conn_01x02_Female, J2 XLR3_Switched, J3 Conn_01x07_Female, J4 Screw_Terminal, U1 ADS1120IRVAR, U2 DS3231M, U3 BME260, U4 ADS1115IRUGT, U5 VO615A

Commit message: update
Parts:
- added H1, H2: MountingHole_Pad, MountingHole:MountingHole_3.2mm_M3, symbol Mechanical:MountingHole_Pad
Changed lines of the file:
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@@
+    )
+  )
+  (symbol (lib_id "Mechanical:MountingHole_Pad") (at 25.4 20.32 0) (unit 1)
+    (in_bom yes) (on_board yes) (dnp no) (fields_autoplaced)
+    (property "Reference" "H1" (at 27.94 18.4063 0)
+      (effects (font (size 1.27 1.27)) (justify left))
+    )
+    (property "Value" "MountingHole_Pad" (at 27.94 20.3273 0)
+      (effects (font (size 1.27 1.27)) (justify left))
+    )
+    (property "Footprint" "MountingHole:MountingHole_3.2mm_M3" (at 25.4 20.32 0)
+      (effects (font (size 1.27 1.27)) hide)
+    )
+    (property "Datasheet" "~" (at 25.4 20.32 0)
+      (effects (font (size 1.27 1.27)) hide)
+    )
+    (pin "1")
+    (instances
+      (project "smart penetrometer"
+        (path "/4bd690aa-2164-4561-b480-04505132937c"
+          (reference "H1") (unit 1)
+        )
+      )
     )
   )
@@
         )
       )
+    )
+  )
+  (symbol (lib_id "Mechanical:MountingHole_Pad") (at 49.53 20.32 0) (unit 1)
+    (in_bom yes) (on_board yes) (dnp no) (fields_autoplaced)
+    (property "Reference" "H2" (at 52.07 18.4063 0)
+      (effects (font (size 1.27 1.27)) (justify left))
+    )
+    (property "Value" "MountingHole_Pad" (at 52.07 20.3273 0)
+      (effects (font (size 1.27 1.27)) (justify left))
+    )
+    (property "Footprint" "MountingHole:MountingHole_3.2mm_M3" (at 49.53 20.32 0)
+      (effects (font (size 1.27 1.27)) hide)
+    )
+    (property "Datasheet" "~" (at 49.53 20.32 0)
+      (effects (font (size 1.27 1.27)) hide)
+    )
+    (pin "1")
+    (instances
+      (project "smart penetrometer"
+        (path "/4bd690aa-2164-4561-b480-04505132937c"
+          (reference "H2") (unit 1)
+        )
+      )

Commit message: pcb and cad update
Parts:
- added J5: Conn_02x04, Connector_PinSocket_2.54mm:PinSocket_2x04_P2.54mm_Vertical, symbol Connector_Generic_MountingPin:Conn_02x04_Odd_Even_MountingPin
- H1, H2: footprint MountingHole:MountingHole_3.2mm_M3 -> MountingHole:MountingHole_3.2mm_M3_Pad
Connections:
- net 3V3: now also J5.2 (Pin_2)
- net CLK: now also J5.5 (Pin_5)
- net GND: now also H1.1, H2.1, J5.1 (Pin_1)
- net MISO: now also J5.7 (Pin_7)
- net MOSI: now also J5.6 (Pin_6)
- net CSN: now reaches A1.10 (D7)
- net CSN: now also J5.4 (Pin_4)
- net CE: now reaches A1.9 (D6)
- net CE: now also J5.3 (Pin_3)
Other:
- note added: "RF Pin"
Changed lines of the file:
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@@
   (no_connect (at 91.44 151.13))
   (no_connect (at 231.14 152.4))
-  (no_connect (at 143.51 111.76))
+  (no_connect (at 74.93 187.96))
   (no_connect (at 88.9 53.34))
   (no_connect (at 55.88 153.67))
   (no_connect (at 168.91 99.06))
   (no_connect (at 251.46 152.4))
+  (no_connect (at 68.58 193.04))
   (no_connect (at 168.91 129.54))
   (no_connect (at 143.51 106.68))
   (no_connect (at 168.91 116.84))
-  (no_connect (at 143.51 114.3))
   (no_connect (at 168.91 106.68))
   (no_connect (at 143.51 109.22))
@@
     (stroke (width 0) (type default))
   )
+  (rectangle (start 50.8 172.72) (end 86.36 194.31)
+    (stroke (width 0) (type default))
+    (fill (type none))
+  )
   (text "THERMOCOUPLE AMPLIFIER" (at 40.64 115.57 0)
     (effects (font (size 1.27 1.27)) (justify left bottom))
@@
     (effects (font (size 1.27 1.27)) (justify left bottom))
   )
+  (text "RF Pin" (at 66.04 175.26 0)
+    (effects (font (size 1.27 1.27)) (justify left bottom))
+  )
   (text "CONNECTORS" (at 149.86 168.91 0)
     (effects (font (size 1.27 1.27)) (justify left bottom))
@@
     )
   )
+  (global_label "CSN" (shape input) (at 143.51 114.3 180) (fields_autoplaced)
+    (effects (font (size 1.27 1.27)) (justify right))
+    (property "Intersheetrefs" "${INTERSHEET_REFS}" (at 136.7942 114.3 0)
+      (effects (font (size 1.27 1.27)) (justify right) hide)
+    )
+  )
   (global_label "3V3" (shape input) (at 40.64 134.62 90) (fields_autoplaced)
     (effects (font (size 1.27 1.27)) (justify left))
@@
     )
   )
+  (global_label "CLK" (shape input) (at 62.23 185.42 180) (fields_autoplaced)
+    (effects (font (size 1.27 1.27)) (justify right))
+    (property "Intersheetrefs" "${INTERSHEET_REFS}" (at 55.7561 185.42 0)
+      (effects (font (size 1.27 1.27)) (justify right) hide)
+    )
+  )
   (global_label "MOSI" (shape input) (at 237.49 38.1 180) (fields_autoplaced)
     (effects (font (size 1.27 1.27)) (justify right))
@@
     )
   )
+  (global_label "MISO" (shape output) (at 62.23 187.96 180) (fields_autoplaced)
+    (effects (font (size 1.27 1.27)) (justify right))
+    (property "Intersheetrefs" "${INTERSHEET_REFS}" (at 54.728 187.96 0)
+      (effects (font (size 1.27 1.27)) (justify right) hide)
+    )
+  )
+  (global_label "CSN" (shape input) (at 74.93 182.88 0) (fields_autoplaced)
+    (effects (font (size 1.27 1.27)) (justify left))
+    (property "Intersheetrefs" "${INTERSHEET_REFS}" (at 81.6458 182.88 0)
+      (effects (font (size 1.27 1.27)) (justify left) hide)
+    )
+  )
   (global_label "GEO_AMP_0" (shape input) (at 251.46 144.78 0) (fields_autoplaced)
     (effects (font (size 1.27 1.27)) (justify left))
@@
     )
   )
+  (global_label "CE" (shape input) (at 62.23 182.88 180) (fields_autoplaced)
+    (effects (font (size 1.27 1.27)) (justify right))
+    (property "Intersheetrefs" "${INTERSHEET_REFS}" (at 56.9052 182.88 0)
+      (effects (font (size 1.27 1.27)) (justify right) hide)
+    )
+  )
   (global_label "SCL" (shape input) (at 231.14 147.32 180) (fields_autoplaced)
     (effects (font (size 1.27 1.27)) (justify right))
@@
     )
   )
+  (global_label "MOSI" (shape input) (at 74.93 185.42 0) (fields_autoplaced)
+    (effects (font (size 1.27 1.27)) (justify left))
+    (property "Intersheetrefs" "${INTERSHEET_REFS}" (at 81.9393 185.3406 0)
+      (effects (font (size 1.27 1.27)) (justify left) hide)
+    )
+  )
   (global_label "3V3" (shape input) (at 247.65 29.21 90) (fields_autoplaced)
     (effects (font (size 1.27 1.27)) (justify left))
@@
     )
   )
+  (global_label "CE" (shape input) (at 143.51 111.76 180) (fields_autoplaced)
+    (effects (font (size 1.27 1.27)) (justify right))
+    (property "Intersheetrefs" "${INTERSHEET_REFS}" (at 138.1852 111.76 0)
+      (effects (font (size 1.27 1.27)) (justify right) hide)
+    )
+  )
   (global_label "3V3" (shape output) (at 158.75 86.36 90) (fields_autoplaced)
     (effects (font (size 1.27 1.27)) (justify left))
@@
     (effects (font (size 1.27 1.27)) (justify left))
     (property "Intersheetrefs" "${INTERSHEET_REFS}" (at 144.7006 168.674 90)
+      (effects (font (size 1.27 1.27)) (justify left) hide)
+    )
+  )
+  (global_label "3V3" (shape input) (at 74.93 180.34 0) (fields_autoplaced)
+    (effects (font (size 1.27 1.27)) (justify left))
+    (property "Intersheetrefs" "${INTERSHEET_REFS}" (at 81.3434 180.34 0)
       (effects (font (size 1.27 1.27)) (justify left) hide)
     )
@@
         (path "/4bd690aa-2164-4561-b480-04505132937c"
           (reference "#PWR020") (unit 1)
+        )
+      )
+    )
+  )
+  (symbol (lib_id "power:GND") (at 49.53 22.86 0) (unit 1)
+    (in_bom yes) (on_board yes) (dnp no)
+    (property "Reference" "#PWR023" (at 49.53 29.21 0)
+      (effects (font (size 1.27 1.27)) hide)
+    )
+    (property "Value" "GND" (at 53.34 25.4 0)
+      (effects (font (size 1.27 1.27)))
+    )
+    (property "Footprint" "" (at 49.53 22.86 0)
+      (effects (font (size 1.27 1.27)) hide)
+    )
+    (property "Datasheet" "" (at 49.53 22.86 0)
+      (effects (font (size 1.27 1.27)) hide)
+    )
+    (pin "1")
+    (instances
+      (project "smart penetrometer"
+        (path "/4bd690aa-2164-4561-b480-04505132937c"
+          (reference "#PWR023") (unit 1)
         )
       )
@@
         (path "/4bd690aa-2164-4561-b480-04505132937c"
           (reference "#PWR0101") (unit 1)
+        )
+      )
+    )
+  )
+  (symbol (lib_id "Connector_Generic_MountingPin:Conn_02x04_Odd_Even_MountingPin") (at 67.31 182.88 0) (unit 1)
+    (in_bom yes) (on_board yes) (dnp no)
+    (property "Reference" "J5" (at 68.58 184.15 0)
+      (effects (font (size 1.27 1.27)))
+    )
+    (property "Value" "Conn_02x04" (at 68.58 177.8 0)
+      (effects (font (size 1.27 1.27)))
+    )
+    (property "Footprint" "Connector_PinSocket_2.54mm:PinSocket_2x04_P2.54mm_Vertical" (at 67.31 182.88 0)
+      (effects (font (size 1.27 1.27)) hide)
+    )
+    (property "Datasheet" "~" (at 67.31 182.88 0)
+      (effects (font (size 1.27 1.27)) hide)
+    )
+    (pin "1")
+    (pin "2")
+    (pin "3")
+    (pin "4")
+    (pin "5")
+    (pin "6")
+    (pin "7")
+    (pin "8")
+    (pin "MP")
+    (instances
+      (project "smart penetrometer"
+        (path "/4bd690aa-2164-4561-b480-04505132937c"
+          (reference "J5") (unit 1)
         )
       )
@@
     )
   )
+  (symbol (lib_id "power:GND") (at 25.4 22.86 0) (unit 1)
+    (in_bom yes) (on_board yes) (dnp no)
+    (property "Reference" "#PWR022" (at 25.4 29.21 0)
+      (effects (font (size 1.27 1.27)) hide)
+    )
+    (property "Value" "GND" (at 29.21 25.4 0)
+      (effects (font (size 1.27 1.27)))
+    )
+    (property "Footprint" "" (at 25.4 22.86 0)
+      (effects (font (size 1.27 1.27)) hide)
+    )
+    (property "Datasheet" "" (at 25.4 22.86 0)
+      (effects (font (size 1.27 1.27)) hide)
+    )
+    (pin "1")
+    (instances
+      (project "smart penetrometer"
+        (path "/4bd690aa-2164-4561-b480-04505132937c"
+          (reference "#PWR022") (unit 1)
+        )
+      )
+    )
+  )
   (symbol (lib_id "power:GND") (at 78.74 132.08 0) (unit 1)
     (in_bom yes) (on_board yes) (dnp no)
@@
   )
   (symbol (lib_id "Mechanical:MountingHole_Pad") (at 25.4 20.32 0) (unit 1)
-    (in_bom yes) (on_board yes) (dnp no) (fields_autoplaced)
-    (property "Reference" "H1" (at 27.94 18.4063 0)
+    (in_bom yes) (on_board yes) (dnp no)
+    (property "Reference" "H1" (at 35.56 17.78 0)
       (effects (font (size 1.27 1.27)) (justify left))
     )
@@
       (effects (font (size 1.27 1.27)) (justify left))
     )
-    (property "Footprint" "MountingHole:MountingHole_3.2mm_M3" (at 25.4 20.32 0)
+    (property "Footprint" "MountingHole:MountingHole_3.2mm_M3_Pad" (at 25.4 20.32 0)
       (effects (font (size 1.27 1.27)) hide)
     )
@@
   )
   (symbol (lib_id "Mechanical:MountingHole_Pad") (at 49.53 20.32 0) (unit 1)
-    (in_bom yes) (on_board yes) (dnp no) (fields_autoplaced)
-    (property "Reference" "H2" (at 52.07 18.4063 0)
+    (in_bom yes) (on_board yes) (dnp no)
+    (property "Reference" "H2" (at 58.42 17.78 0)
       (effects (font (size 1.27 1.27)) (justify left))
     )
@@
       (effects (font (size 1.27 1.27)) (justify left))
     )
-    (property "Footprint" "MountingHole:MountingHole_3.2mm_M3" (at 49.53 20.32 0)
+    (property "Footprint" "MountingHole:MountingHole_3.2mm_M3_Pad" (at 49.53 20.32 0)
       (effects (font (size 1.27 1.27)) hide)
     )
@@
         )
       )
+    )
+  )
+  (symbol (lib_id "power:GND") (at 62.23 180.34 270) (unit 1)
+    (in_bom yes) (on_board yes) (dnp no)
+    (property "Reference" "#PWR021" (at 55.88 180.34 0)
+      (effects (font (size 1.27 1.27)) hide)
+    )
+    (property "Value" "GND" (at 57.15 180.34 90)
+      (effects (font (size 1.27 1.27)))
+    )
+    (property "Footprint" "" (at 62.23 180.34 0)
+      (effects (font (size 1.27 1.27)) hide)
+    )
+    (property "Datasheet" "" (at 62.23 180.34 0)
+      (effects (font (size 1.27 1.27)) hide)
+    )
+    (pin "1")
+    (instances
+      (project "smart penetrometer"
+        (path "/4bd690aa-2164-4561-b480-04505132937c"
+          (reference "#PWR021") (unit 1)
+        )
+      )

Commit message: PCB update
Parts:
- removed U4: ADS1115IRUGT, kitest:10X2QFN, symbol Analog_ADC:ADS1115IDGS
- U1: footprint Package_DFN_QFN:VQFN-16-1EP_3x3mm_P0.5mm_EP1.45x1.45mm_ThermalVias -> kitest:ADS1120IPW 16TSSOP
Connections:
- net 3V3: now also U1.12 (AVDD), U1.13 (DVDD); no longer U1.10 (AVDD), U1.11 (DVDD)
- net CLK: now also U1.1 (SCLK); no longer U1.15 (SCLK)
- net GEO_AMP_0: now also U1.7 (AIN2)
- net GEO_AMP_1: now also U1.6 (AIN3/REFN1)
- net GND: now also U1.4 (DGND), U1.5 (AVSS); no longer U1.1 (CLK), U1.17 (thermal), U1.2 (DGND)
- net MISO: now also U1.15 (DOUT/~{DRDY}); no longer U1.13 (DOUT/~{DRDY})
- net MOSI: now also U1.16 (DIN); no longer U1.14 (DIN)
- net TEMP_AMP_CS: now also U1.2 (~{CS}); no longer U1.16 (~{CS})
- net at C1.2, C2.1, R3.1: now also U1.11 (AIN0/REFP1); no longer U1.9 (AIN0/REFP1)
- net at C2.2, C3.1, R4.1: now also U1.10 (AIN1); no longer U1.8 (AIN1)
- no-connect marks 29 -> 23
Other:
- note removed: "GEOPHONE ADC W/ AMPLIFIER"
- moved on the sheet: J5

Commit message: PCB update
Parts:
- added C10: C_0.1uF, Capacitor_SMD:C_1206_3216Metric, symbol Device:C_Small
- added C7: CDIF2_100nF, Capacitor_SMD:C_1206_3216Metric, symbol Device:C_Small
- added C8: CCM4_10nf, Capacitor_SMD:C_1206_3216Metric, symbol Device:C_Small
- added C9: CCM3_10nF, Capacitor_SMD:C_1206_3216Metric, symbol Device:C_Small
- added R10, R11, R8, R9: R_47, Resistor_SMD:R_1206_3216Metric, symbol Device:R_Small_US
- added R12: RF4_1K, Resistor_SMD:R_1206_3216Metric, symbol Device:R_Small_US
- added R13: RF3_1K, Resistor_SMD:R_1206_3216Metric, symbol Device:R_Small_US
- added R14: RREF_3.3K, Resistor_SMD:R_1206_3216Metric, symbol Device:R_Small_US
- added R15: RF1_1K, Resistor_SMD:R_1206_3216Metric, symbol Device:R_Small_US
- added R16: RF2_1K, Resistor_SMD:R_1206_3216Metric, symbol Device:R_Small_US
- added R17: R_1K, Resistor_SMD:R_1206_3216Metric, symbol Device:R_Small_US
- added R18, R19, R20, R21: R_50, Resistor_SMD:R_1206_3216Metric, symbol Device:R_Small_US
- added U4: ADS1118IDGS, kitest:ADS1118_10VSSOP, symbol Analog_ADC:ADS1118IDGS
- C1: value C_0.047uF -> CCM2_10nF
- C2: value C_0.47uF -> CDIF1_100nF
- C3: value C_0.047uF -> CCM1_10nf
- R1: value R_1MOhm -> RLEAD2_3.3K
- R2: value R_1MOhm -> RLEAD1_3.3K
- R3: value R_800Ohm -> RF2_1K
- R4: value R_800Ohm -> RF1_1K
Connections:
- net 3V3: now also C10.1, U4.8 (VDD); no longer R1.1
- net CLK: now also R11.1, R18.1; no longer U1.1 (SCLK)
- net GEO_AMP_0: now also R15.2, R17.1; no longer U1.7 (AIN2)
- net GEO_AMP_1: now also R16.2, R17.2; no longer U1.6 (AIN3/REFN1)
- net GND: no longer C1.1, C3.2, C5.2, R2.2, U1.5 (AVSS)
- net MISO: now also R20.1, R9.1; no longer U1.15 (DOUT/~{DRDY})
- net MOSI: now also R10.1, R19.1; no longer U1.16 (DIN)
- net GEO_CS: now reaches A1.8 (D5)
- net GEO_CS: now also R21.1
- net at U1.8 (REFN0): now also C7.2, C8.1, R12.2
- net at U1.9 (REFP0): now also C7.1, C9.2, R13.2
- net TEMP_AMP_0 renamed RTD_1
- net RTD_1: no longer R3.2
- net TEMP_AMP_1 renamed RTD_2
- net RTD_2: no longer R4.2
- net TEMP_AMP_CS: no longer names the net of U1.2 (~{CS})
- net TEMP_AMP_CS: now also R8.2; no longer A1.12 (D9)
- new net: R9.2, U1.15 (DOUT/~{DRDY})
- new net: R18.2, U4.1 (SCLK)
- new net: R19.2, U4.10 (DIN)
- new net: R21.2, U4.2 (~{CS})
- new net: R15.1, U4.4 (AIN0)
- new net: R16.1, U4.5 (AIN1)
- new net: R20.2, U4.9 (DOUT/~{DRDY})
- new net: R1.1, R13.1, R14.2, R3.2
- new net: R2.2, R4.2, U1.6 (AIN3/REFN1)
- new net: R11.2, U1.1 (SCLK)
- new net: R10.2, U1.16 (DIN)
- new net GNDA: C1.1, C10.2, C3.2, C5.2, C8.2, C9.1, R12.1, R14.1, U1.5 (AVSS), U4.3 (GND)
- new net RTD_CS: A1.12 (D9), R8.1
Other:
- moved on the sheet: A1, C1, C2, C3, C4, C5, H1, H2, J1, J2A, J4, R1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

Commit message: pcb update
Connections:
- net 3V3: now also J2.2
- net VIN: no longer J2.2
Changed lines of the file:
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@@
     )
   )
-  (global_label "VIN" (shape output) (at 100.965 42.545 0) (fields_autoplaced)
+  (global_label "3V3" (shape output) (at 100.965 42.545 0) (fields_autoplaced)
     (effects (font (size 1.27 1.27)) (justify left))
-    (property "Intersheetrefs" "${INTERSHEET_REFS}" (at 106.4019 42.4656 0)
+    (property "Intersheetrefs" "${INTERSHEET_REFS}" (at 107.3784 42.545 0)
       (effects (font (size 1.27 1.27)) (justify left) hide)
     )
@@
     )
   )
-  (global_label "3V3" (shape output) (at 176.53 85.09 90) (fields_autoplaced)
+  (global_label "3V3" (shape input) (at 176.53 85.09 90) (fields_autoplaced)
     (effects (font (size 1.27 1.27)) (justify left))
-    (property "Intersheetrefs" "${INTERSHEET_REFS}" (at 176.4506 79.1693 90)
+    (property "Intersheetrefs" "${INTERSHEET_REFS}" (at 176.53 78.6766 90)
       (effects (font (size 1.27 1.27)) (justify left) hide)
     )

Commit message: PCB update
Parts:
- removed C5: C_0.1uF, Capacitor_SMD:C_1206_3216Metric, symbol Device:C_Small
- removed C7: CDIF2_100nF, Capacitor_SMD:C_1206_3216Metric, symbol Device:C_Small
- removed C8: CCM4_10nf, Capacitor_SMD:C_1206_3216Metric, symbol Device:C_Small
- removed C9: CCM3_10nF, Capacitor_SMD:C_1206_3216Metric, symbol Device:C_Small
- removed J2: XLR3_Switched, kitest:grounded_switch, symbol Connector:XLR3_Switched
- removed R1: RLEAD2_3.3K, Resistor_SMD:R_1206_3216Metric, symbol Device:R_Small_US
- removed R10, R8, R9: R_47, Resistor_SMD:R_1206_3216Metric, symbol Device:R_Small_US
- removed R12: RF4_1K, Resistor_SMD:R_1206_3216Metric, symbol Device:R_Small_US
- removed R13: RF3_1K, Resistor_SMD:R_1206_3216Metric, symbol Device:R_Small_US
- removed R14: RREF_3.3K, Resistor_SMD:R_1206_3216Metric, symbol Device:R_Small_US
- removed R2: RLEAD1_3.3K, Resistor_SMD:R_1206_3216Metric, symbol Device:R_Small_US
- removed R3: RF2_1K, Resistor_SMD:R_1206_3216Metric, symbol Device:R_Small_US
- removed R4: RF1_1K, Resistor_SMD:R_1206_3216Metric, symbol Device:R_Small_US
- removed U1: ADS1120IRVAR, kitest:ADS1120IPW 16TSSOP, symbol Analog_ADC:ADS1120-PW
- added C6: C_1uF, Capacitor_SMD:C_1206_3216Metric, symbol Device:C_Small
- added J3: Conn_01x02, Connector_PinSocket_2.54mm:PinSocket_1x02_P2.54mm_Horizontal, symbol Connector:Conn_01x02_Female
- added U2: ADP7157-3.3, Package_SO:SOIC-8-1EP_3.9x4.9mm_P1.27mm_EP2.29x3mm, symbol Regulator_Linear:ADP7142ARDZ-3.3
- C1: value CCM2_10nF -> C_10uF
- C2: value CDIF1_100nF -> C_1uF
- C3: value CCM1_10nf -> C_1uF
- C4: value C_0.1uF -> C_10uF
- J2: renamed from J1; value Conn_01x02_Female -> Conn_01x02
- R11: value R_47 -> R_10K
- renumbered C10 to C5, C6 to C7, J4 to J1, J3 to J4, R17 to R1, R6 to R10, R15 to R2, R16 to R3, R7 to R4, R18 to R5, R19 to R6, R20 to R7, R21 to R8, R5 to R9, U5 to U1, U4 to U3, U2 to U4, U3 to U5
Connections:
- net RTD_1 is gone; now on net RTD: J4.2 (Pin_2)
- net RTD_2 is gone; now on net 3V3: J4.1 (Pin_1)
- net 3V3: now also A1.11 (D8), A1.18 (AREF), U1.4, U2.1 (VOUT), U2.2 (VOUT)
- net CLK: no longer R11.1
- net GND: now also C1.2, C2.2, C3.2, C6.2, U2.9 (GND); no longer A1.4 (GND)
- net GNDA: now also A1.4 (GND), R11.2; no longer C1.1, C3.2
- net at C2.1: now also U2.7 (VREG); no longer C1.2
- net RTD: now reaches A1.20 (A1)
- net RTD: now also R11.1
- net at C3.1: now also U2.5 (REF_S), U2.6 (REF); no longer C2.2
- net +3V3 renamed +BATT
- net +BATT: now also J3.1 (Pin_1)
- removed net 5V0: A1.11 (D8), A1.27 (+5V), U1.4
- net VIN: no longer names the net of A1.30 (VIN)
- new net: C6.1, U2.3 (BYP)
- new net BATT: C1.1, J3.2 (Pin_2), U2.4 (EN), U2.8 (VIN)
- no-connect marks 23 -> 20
Other:
- note added: "3V3 VOLTAGE REGULATOR"
- note added: "GEOPGONE AMPLIFIER"
- note removed: "SWITCH"
- note removed: "THERMOCOUPLE AMPLIFIER"
- moved on the sheet: J2, J4
