File: V0/V0.6/V0.6.0/hardware_design/PCB/smart penetrometer/smart penetrometer.kicad_pcb (KiCad board)
At the start: 4 copper layers, 29 x 93 mm, 35 parts, among them J1 Screw_Terminal, J2 Conn_01x02, J3 Conn_01x02, J4 Conn_01x07_Female, J5 Conn_02x04, U1 VO615A, U2 ADP7157-3.3, U3 ADS1118IDGS, U4 DS3231M, U5 BME260

Commit message: correction
Parts:
- removed C1, C4: C_10uF, Capacitor_SMD:C_1206_3216Metric
- removed C3: C_1uF, Capacitor_SMD:C_1206_3216Metric
- removed J1: Screw_Terminal, TerminalBlock:TerminalBlock_bornier-2_P5.08mm
- removed R4: R_1.9kOhm, Resistor_SMD:R_1206_3216Metric
- removed U1: VO615A, footprints:Vishay_VOS615A
- added D2: SMZ1_770mV, Diode_SMD:D_MELF, B.Cu at (170.5, 136.0)
- added G***: LOGO, kitest:uofsc_logo_1in, B.Cu at (177.3, 79.6)
- added JP1: Jumper_2, Connector_PinHeader_2.54mm:PinHeader_1x02_P2.54mm_Vertical, F.Cu at (188.2, 123.3)
- added JP2: Jumper_3, Connector_PinHeader_2.54mm:PinHeader_1x03_P2.54mm_Vertical, F.Cu at (166.4, 75.8)
- added U6: LM321, Package_TO_SOT_SMD:SOT-23-5, B.Cu at (165.9, 139.1)
- A1: value Arduino_Nano_v3.x -> Arduino Nano
- R1: value R_1K -> R_7.5K
- R2: value RF1_1K -> R_32k
- R3: value RF2_1K -> R_100
- U2: value ADP7157-3.3 -> ADP124ARHZ-3.3-R7; footprint Package_SO:SOIC-8-1EP_3.9x4.9mm_P1.27mm_EP2.29x3mm -> footprint:RH_8_1_ADI
- U5: footprint kitest:TDS_module -> kitest:BME260
- moved R3 13.3 mm to (180.4, 139.1), turned to 180 degrees
- moved J2 9.72 mm to (164.9, 63.1), turned to 90 degrees
- moved J3 9.47 mm to (167.4, 66.4), turned to -90 degrees
- moved R1 3.60 mm to (166.4, 142.6), turned to 0 degrees
- moved R2 3.45 mm to (166.4, 135.3), turned to 0 degrees
- moved R11 2.79 mm to (188.8, 115.7), turned to 90 degrees
- moved R8 1.55 mm to (175.0, 133.7), turned to -90 degrees
- moved G*** 0.76 mm to (177.6, 57.5)
Connections:
- A1 pad 11: 3V3 -> Vtrig
- A1 pad 17: 3V3 -> Net-(A1-3V3)
- A1 pad 27: unconnected-(A1-+5V-Pad27) -> 5V0
- C2 pad 1: Net-(U2-VREG) -> Net-(JP2-C)
- C5 pad 2: GNDA -> GND
- C6 pad 1: Net-(U2-BYP) -> 3V3
- J4 pad 3: GEO_AMP_0 -> GEOPHONE
- J4 pad 4: GEO_AMP_1 -> GNDA
- R1 pad 1: GEO_AMP_0 -> Net-(U6--)
- R1 pad 2: GEO_AMP_1 -> GNDA
- R2 pad 2: GEO_AMP_0 -> Net-(U6--)
- R3 pad 1: Net-(U3-AIN1) -> GEOPHONE
- R3 pad 2: GEO_AMP_1 -> Net-(D2-K)
- U2 pad 3: Net-(U2-BYP) -> 3V3
- U2 pad 4: BATT -> GND
- U2 pad 5: Net-(U2-REF) -> Net-(JP2-C)
- U2 pad 6: Net-(U2-REF) -> unconnected-(U2-NC-Pad6)
- U2 pad 7: Net-(U2-VREG) -> Net-(JP2-C)
- U2 pad 8: BATT -> Net-(JP2-C)
- U3 pad 3: GNDA -> GND
- U3 pad 5: Net-(U3-AIN1) -> unconnected-(U3-AIN1-Pad5)
Routing:
- net 5V0: track 0.00 -> 36.0 mm
- net BATT: track 28.4 -> 4.95 mm, vias 1 -> 0
- net Net-(JP2-C): track 0.00 -> 18.7 mm
- net GEO_AMP_1: track 16.2 -> 0.00 mm
- net Net-(D2-K): track 0.00 -> 14.6 mm
- net GEO_AMP_0: track 13.3 -> 0.00 mm
- net GND: track 14.2 -> 26.9 mm, vias 31 -> 35
- net Net-(U3-AIN1): track 12.3 -> 0.00 mm
- net Net-(J1-Pin_2): track 11.0 -> 0.00 mm
- net Net-(U2-BYP): track 9.73 -> 0.00 mm
- net 3V3: track 12.3 -> 21.6 mm
- net Net-(U6--): track 0.00 -> 8.58 mm
- net Net-(U3-AIN0): track 9.58 -> 18.1 mm
- net GEOPHONE: track 0.00 -> 7.99 mm
- net GNDA: track 5.15 -> 11.0 mm, vias 3 -> 2
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Other:
- board text added: "BAT"
- board text added: "BY MALICHI FLEMMING II 04/01/2024"
- board text added: "CE"
- board text added: "CLK"
- board text added: "CSN"
- board text added: "MISO"
- board text added: "MOSI"
- board text added: "RTD"
- board text added: "SPECIES V0.6.0"
- board text added: "USB"
- board text removed: "BY MALICHI FLEMMING II 11/25/2023"
- board text removed: "OPTOCOUPLER"
- board text removed: "SPECIES V0.5.1"
- board text removed: "TERMINALS"
- board text removed: "THERMO"
