File: V0/V0.6/V0.6.0/hardware_design/PCB/smart penetrometer/smart penetrometer.kicad_pcb (KiCad board)
At the start: 4 copper layers, 29 x 93 mm, 34 parts, among them J2 Conn_01x02, J3 Conn_01x02, J4 Conn_01x07_Female, J5 Conn_02x04, U2 ADP124ARHZ-3.3-R7, U3 ADS1118IDGS, U4 DS3231M, U5 BME260, U6 LM321

Commit message: Update smart penetrometer.kicad_pcb
Other:
- board size 29 x 93 mm -> 29 x 93.3 mm
- board text added: "BATTERY"
- board text added: "X"
- board text removed: "BATT"
Changed lines of the file:
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@@
     )
     (pad_to_mask_clearance 0)
-    (grid_origin 172.5 131.19)
+    (grid_origin 172.5 0)
     (pcbplotparams
       (layerselection 0x00010fc_ffffffff)
@@
     (property "ki_keywords" "connector")
     (attr through_hole)
-    (fp_text reference "J4" (at -0.462 17.59 180) (layer "F.SilkS")
+    (fp_text reference "J4" (at -0.138 -2.5 180) (layer "F.SilkS")
         (effects (font (size 1 1) (thickness 0.15)))
     )
@@
     (property "ki_keywords" "battery cell")
     (attr smd)
-    (fp_text reference "BT1" (at -0.254 -6.35 180) (layer "F.SilkS")
+    (fp_text reference "BT1" (at -0.05 -5.19 180) (layer "F.SilkS")
         (effects (font (size 1 1) (thickness 0.25) bold))
     )
@@
     (property "ki_keywords" "Jumper SPDT")
     (attr through_hole)
-    (fp_text reference "JP2" (at -3.048 2.54) (layer "F.SilkS")
+    (fp_text reference "JP2" (at 0.094 -2.452) (layer "F.SilkS")
         (effects (font (size 1 1) (thickness 0.15)))
     )
@@
         (effects (font (size 1 1) (thickness 0.15)))
     )
-    (fp_text user "USB" (at 7.62 36.607 unlocked) (layer "F.SilkS")
-        (effects (font (size 1 1) (thickness 0.15)))
-    )
     (fp_text user "${REFERENCE}" (at 6.35 19.05 90) (layer "F.Fab")
         (effects (font (size 1 1) (thickness 0.15)))
@@
     )
   )
+  (gr_line (start 169.831856 67.112593) (end 173.131856 67.112593)
+    (stroke (width 0.1) (type default)) (layer "F.SilkS"))
+  (gr_arc (start 169.831856 67.112593) (mid 169.4 66.933712) (end 169.221119 66.501856)
+    (stroke (width 0.1) (type default)) (layer "F.SilkS"))
+  (gr_arc (start 174.070737 63.03) (mid 173.891856 63.461856) (end 173.46 63.640737)
+    (stroke (width 0.1) (type default)) (layer "F.SilkS"))
+  (gr_arc (start 169.5 63.64) (mid 169.068144 63.461119) (end 168.889263 63.029263)
+    (stroke (width 0.1) (type default)) (layer "F.SilkS"))
+  (gr_arc (start 173.742593 66.502593) (mid 173.563712 66.934449) (end 173.131856 67.11333)
+    (stroke (width 0.1) (type default)) (layer "F.SilkS"))
+  (gr_line (start 169.5 63.64) (end 173.46 63.64)
+    (stroke (width 0.1) (type default)) (layer "F.SilkS"))
+  (gr_arc (start 173.46 62.419263) (mid 173.891856 62.598144) (end 174.070737 63.03)
+    (stroke (width 0.1) (type default)) (layer "F.SilkS"))
   (gr_line (start 179.04 143.872) (end 179.04 140.7)
     (stroke (width 0.15) (type solid)) (layer "F.SilkS"))
+  (gr_line (start 173.131856 65.891856) (end 169.831856 65.891856)
+    (stroke (width 0.1) (type default)) (layer "F.SilkS"))
   (gr_line (start 173.96 143.83) (end 173.96 140.72)
     (stroke (width 0.15) (type solid)) (layer "F.SilkS"))
-  (gr_rect (start 162.814 51.76) (end 191.77 144.78)
-    (stroke (width 0.1) (type solid)) (fill none) (layer "Edge.Cuts"))
-  (gr_text "MOSI" (at 176.818 90.296) (layer "B.SilkS")
+  (gr_line (start 169.5 62.418526) (end 173.46 62.418526)
+    (stroke (width 0.1) (type default)) (layer "F.SilkS"))
+  (gr_arc (start 168.889263 63.029263) (mid 169.068144 62.597407) (end 169.5 62.418526)
+    (stroke (width 0.1) (type default)) (layer "F.SilkS"))
+  (gr_arc (start 169.221119 66.501856) (mid 169.4 66.07) (end 169.831856 65.891119)
+    (stroke (width 0.1) (type default)) (layer "F.SilkS"))
+  (gr_arc (start 173.131856 65.891856) (mid 173.563712 66.070737) (end 173.742593 66.502593)
+    (stroke (width 0.1) (type default)) (layer "F.SilkS"))
+  (gr_arc (start 166.8 145.65) (mid 163.985715 144.484285) (end 162.82 141.67)
+    (stroke (width 0.1) (type default)) (layer "Edge.Cuts"))
+  (gr_line (start 162.82 141.67) (end 162.82 56.299988)
+    (stroke (width 0.1) (type default)) (layer "Edge.Cuts"))
+  (gr_arc (start 187.75 52.319988) (mid 190.592578 53.497422) (end 191.770012 56.34)
+    (stroke (width 0.1) (type default)) (layer "Edge.Cuts"))
+  (gr_line (start 187.75 145.65) (end 166.8 145.65)
+    (stroke (width 0.1) (type default)) (layer "Edge.Cuts"))
+  (gr_line (start 187.75 52.319988) (end 166.8 52.319988)
+    (stroke (width 0.1) (type default)) (layer "Edge.Cuts"))
+  (gr_line (start 191.770012 56.34) (end 191.770012 141.629988)
+    (stroke (width 0.1) (type default)) (layer "Edge.Cuts"))
+  (gr_arc (start 191.770012 141.629988) (mid 190.592578 144.472566) (end 187.75 145.65)
+    (stroke (width 0.1) (type default)) (layer "Edge.Cuts"))
+  (gr_arc (start 162.82 56.299988) (mid 163.985715 53.485703) (end 166.8 52.319988)
+    (stroke (width 0.1) (type default)) (layer "Edge.Cuts"))
+  (gr_text "X" (at 173.58 90.28) (layer "B.SilkS")
+    (effects (font (size 0.75 0.75) (thickness 0.1875) bold) (justify left bottom mirror))
+  )
+  (gr_text "MOSI" (at 176.95 90.26) (layer "B.SilkS")
     (effects (font (size 0.75 0.75) (thickness 0.1875) bold) (justify left bottom mirror))
   )
@@
     (effects (font (size 0.75 0.75) (thickness 0.1875) bold) (justify left bottom))
   )
-  (gr_text "BATT" (at 166.404 61.848) (layer "F.SilkS")
+  (gr_text "BATTERY" (at 169.16 63.51) (layer "F.SilkS")
     (effects (font (size 0.75 0.75) (thickness 0.1875) bold) (justify left bottom))
   )
@@
     (effects (font (size 0.75 0.75) (thickness 0.15)))
   )
-  (gr_text "+" (at 165.134 77.596) (layer "F.SilkS")
+  (gr_text "+" (at 166.92 61.7) (layer "F.SilkS")
     (effects (font (size 0.75 0.75) (thickness 0.1875) bold) (justify left bottom))
   )
@@
     (effects (font (size 0.75 0.75) (thickness 0.1875) bold) (justify left bottom))
   )
-  (gr_text "SWITCH" (at 169.198 66.975) (layer "F.SilkS")
+  (gr_text "SWITCH" (at 169.479856 66.957593) (layer "F.SilkS")
     (effects (font (size 0.75 0.75) (thickness 0.1875) bold) (justify left bottom))
   )
@@
         (xy 162.81 51.76)
         (xy 191.77 51.76)
-        (xy 191.77 144.78)
-        (xy 162.81 144.78)
+        (xy 191.77 146.16)
+        (xy 162.81 146.16)
       )
     )
@@
     (polygon
       (pts
-        (xy 191.77 144.78)
-        (xy 162.814 144.78)
+        (xy 191.77 146.1)
+        (xy 162.814057 146.1)
         (xy 162.81 51.76)
         (xy 191.77 51.76)
@@
     (polygon
       (pts
-        (xy 191.77 144.78)
-        (xy 162.814 144.78)
+        (xy 191.77 146.11)
+        (xy 162.814057 146.11)
         (xy 162.81 51.76)
         (xy 191.77 51.76)
@@
         (xy 162.81 51.76)
         (xy 191.77 51.76)
-        (xy 191.77 144.78)
-        (xy 162.81 144.78)
+        (xy 191.77 146.11)
+        (xy 162.81 146.11)
       )
     )
