File: System_development/Columbia/V0/V0.6/V0.6.0/hardware_design/Base Station/SPECIES_receiver/_autosave-SPECIES_receiver.kicad_sch (KiCad schematic)
At the start: 8 parts, among them J1 Conn_02x04_Odd_Even_MountingP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, J2 Conn_02x04_Odd_Even_MountingP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, J3 Conn_02x20_Odd_Even

Commit message: updated base station receiver pcb
decreased board size, flipped nRF pinout, and added clearer silkscreen labels
Parts:
- removed J3: Conn_02x20_Odd_Even, Connector_PinSocket_2.54mm:PinSocket_2x20_P2.54mm_Vertical, symbol Connector_Generic:Conn_02x20_Odd_Even
- added C4, C5, C6: C_Small, SPECIES_Elongated:C_1206_3216Metric, symbol Device:C_Small
Connections:
- net 3V3: now also C1.1, C2.1, C3.1, J1.2 (Pin_2), J2.2 (Pin_2), C4.1, C5.1, C6.1; no longer J2.8 (Pin_8)
- net CE: now also J1.3 (Pin_3), J2.3 (Pin_3); no longer J2.5 (Pin_5)
- net CLK: now also J1.5 (Pin_5), J2.5 (Pin_5); no longer J2.3 (Pin_3)
- net CSN: now also J1.4 (Pin_4), J2.4 (Pin_4); no longer J2.6 (Pin_6)
- net GND: now also J1.1 (Pin_1), J2.1 (Pin_1), C4.2, C5.2, C6.2; no longer A2.29 (GND), J2.7 (Pin_7)
- net MISO: now also J1.7 (Pin_7), J2.7 (Pin_7); no longer J2.1 (Pin_1)
- net MOSI: now also J1.6 (Pin_6), J2.6 (Pin_6); no longer J2.4 (Pin_4)
- new net: A2.27 (+5V), A2.30 (VIN)
- now unconnected: A1.30 (VIN)
Other:
- company: (none) -> Sydney Morris - ARTS Lab
- title: (none) -> Receiver PCB for Base Station
- moved on the sheet: C1, C2, C3, J1, J2
