File: System_development/Columbia/V0/V0.6/V0.6.1/sensor_node/hardware_design/PCB/smart penetrometer/smart penetrometer.kicad_pcb (KiCad board)
At the start: 4 copper layers, 29 x 93.3 mm, 31 parts, among them J2 Conn_01x02, J3 Conn_01x02, J4 Conn_01x07_Female, J5 Conn_02x04, U1 LM321, U2 ADP124ARHZ-3.3-R7, U4 DS3231M, U5 BME260, U7 ADS1115IDGS

Commit message: V0.6.1 update
Connections:
- R5 pad 1: SCL -> 3V3
- R5 pad 2: Net-(U7-SCL) -> SCL
- R6 pad 1: SDA -> 3V3
- R6 pad 2: Net-(U7-SDA) -> SDA
- U7 pad 10: Net-(U7-SCL) -> SCL
- U7 pad 9: Net-(U7-SDA) -> SDA
Routing:
- net SCL: track 78.9 -> 87.3 mm
- net SDA: track 70.1 -> 77.6 mm
- net Net-(U7-SCL): track 7.16 -> 0.00 mm
- net Net-(U7-SDA): track 5.87 -> 0.00 mm
- net 3V3: track 31.9 -> 35.0 mm, vias 6 -> 7
- net EC_DATA: track 16.2 -> 16.3 mm, vias 0 -> 1
