File: SYS_DEV/Mississippi/v0.1/spike-PCB/spike_PCB.kicad_pcb (KiCad board)
At the start: 2 copper layers, 55.9 x 68.6 mm, 6 parts, among them J1 Power_Input_Screw_Terminal, J2 Sensing_Spike_Screw_Terminal

Commit message: updated two errors on PCB
Connections:
- J2 pad 2: Net-(J2-Pin_2) -> Net-(A1-A3)
- R1 pad 1: Net-(J2-Pin_2) -> Net-(A1-A3)
- R1 pad 2: Net-(A1-A3) -> GND
- RF1 pad 4: unconnected-(RF1-MISO-Pad4) -> Net-(A1-MISO)
- RF1 pad 8: Net-(A1-MISO) -> unconnected-(RF1-IRQ-Pad8)
Routing:
- net GND: track 59.7 -> 75.5 mm
- net Net-(J2-Pin_2): track 8.67 -> 0.00 mm
- net Net-(A1-A3): track 50.2 -> 55.7 mm
- net Net-(A1-MISO): track 81.5 -> 83.4 mm
Other:
- board text added: "Clay Crews 07/25 v0.1.2"
- board text removed: "Clay Crews 01/24"
Changed lines of the file:
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@@
   (net 22 "unconnected-(A1-+5V-Pad27)")
   (net 23 "unconnected-(A1-~{RESET}-Pad28)")
-  (net 24 "unconnected-(RF1-MISO-Pad4)")
+  (net 24 "unconnected-(RF1-IRQ-Pad8)")
   (net 25 "GND")
   (net 26 "Net-(A1-3V3)")
@@
   (net 29 "Net-(A1-SCK)")
   (net 30 "Net-(A1-VIN)")
-  (net 31 "Net-(J2-Pin_2)")
   (footprint "spike_PCB:SD_Card_Module" (layer "F.Cu")
     (at 259.08 175.26 -90)
@@
       (net 26 "Net-(A1-3V3)") (pinfunction "Pin_1") (pintype "passive"))
     (pad "2" thru_hole oval (at 5 0) (size 1.98 3.96) (drill 1.32) (layers "*.Cu" "*.Mask")
-      (net 31 "Net-(J2-Pin_2)") (pinfunction "Pin_2") (pintype "passive"))
+      (net 27 "Net-(A1-A3)") (pinfunction "Pin_2") (pintype "passive"))
     (model "${KICAD6_3DMODEL_DIR}/TerminalBlock.3dshapes/TerminalBlock_Altech_AK300-2_P5.00mm.wrl"
       (offset (xyz 0 0 0))
@@
       (stroke (width 0.1) (type solid)) (layer "F.Fab"))
     (pad "1" thru_hole circle (at 0 0) (size 1.6 1.6) (drill 1) (layers "*.Cu" "*.Mask")
-      (net 31 "Net-(J2-Pin_2)") (pintype "passive"))
-    (pad "2" thru_hole oval (at 7.62 0) (size 1.6 1.6) (drill 1) (layers "*.Cu" "*.Mask")
       (net 27 "Net-(A1-A3)") (pintype "passive"))
+    (pad "2" thru_hole oval (at 7.62 0) (size 1.6 1.6) (drill 1) (layers "*.Cu" "*.Mask")
+      (net 25 "GND") (pintype "passive"))
     (model "${KICAD6_3DMODEL_DIR}/Resistor_THT.3dshapes/R_Axial_DIN0207_L6.3mm_D2.5mm_P7.62mm_Horizontal.wrl"
       (offset (xyz 0 0 0))
@@
       (net 29 "Net-(A1-SCK)") (pinfunction "SCK") (pintype "input"))
     (pad "4" thru_hole circle (at 0 7.62 90) (size 1.6 1.6) (drill 1) (layers "*.Cu" "*.Mask")
-      (net 24 "unconnected-(RF1-MISO-Pad4)") (pinfunction "MISO") (pintype "output+no_connect"))
+      (net 13 "Net-(A1-MISO)") (pinfunction "MISO") (pintype "output"))
     (pad "5" thru_hole circle (at 2.54 0 90) (size 1.6 1.6) (drill 1) (layers "*.Cu" "*.Mask")
       (net 26 "Net-(A1-3V3)") (pinfunction "VCC") (pintype "power_in"))
@@
       (net 28 "Net-(A1-MOSI)") (pinfunction "MOSI") (pintype "input"))
     (pad "8" thru_hole circle (at 2.54 7.62 90) (size 1.6 1.6) (drill 1) (layers "*.Cu" "*.Mask")
-      (net 13 "Net-(A1-MISO)") (pinfunction "IRQ") (pintype "input"))
+      (net 24 "unconnected-(RF1-IRQ-Pad8)") (pinfunction "IRQ") (pintype "input+no_connect"))
   )
   (gr_poly
@@
     )
     (stroke (width 0.1) (type solid)) (fill none) (layer "Edge.Cuts"))
-  (gr_text "Clay Crews\n01/24" (at 218.44 160.02 90) (layer "B.SilkS")
+  (gr_text "Clay Crews\n07/25 v0.1.2" (at 218.44 160.02 90) (layer "B.SilkS")
     (effects (font (size 1 1) (thickness 0.15)) (justify bottom mirror))
   )
@@
   (segment (start 251.46 157.48) (end 236.22 142.24) (width 0.25) (layer "F.Cu") (net 12))
   (segment (start 248.92 176.39137) (end 253.31863 180.79) (width 0.25) (layer "F.Cu") (net 13))
-  (segment (start 264.61 165.55) (end 256.54 157.48) (width 0.25) (layer "F.Cu") (net 13))
   (segment (start 264.61 180.526396) (end 264.61 165.55) (width 0.25) (layer "F.Cu") (net 13))
   (segment (start 256.54 157.48) (end 236.22 137.16) (width 0.25) (layer "F.Cu") (net 13))
   (segment (start 248.92 175.26) (end 248.92 176.39137) (width 0.25) (layer "F.Cu") (net 13))
-  (segment (start 256.54 165.1) (end 256.54 157.48) (width 0.25) (layer "F.Cu") (net 13))
   (segment (start 264.346396 180.79) (end 264.61 180.526396) (width 0.25) (layer "F.Cu") (net 13))
+  (segment (start 257.683 158.623) (end 256.54 157.48) (width 0.25) (layer "F.Cu") (net 13))
   (segment (start 253.31863 180.79) (end 264.346396 180.79) (width 0.25) (layer "F.Cu") (net 13))
+  (segment (start 257.683 166.497) (end 256.54 167.64) (width 0.25) (layer "F.Cu") (net 13))
+  (segment (start 264.61 165.55) (end 257.683 158.623) (width 0.25) (layer "F.Cu") (net 13))
+  (segment (start 257.683 158.623) (end 257.683 166.497) (width 0.25) (layer "F.Cu") (net 13))
   (segment (start 243.84 175.26) (end 226.06 175.26) (width 0.25) (layer "F.Cu") (net 25))
   (segment (start 241.3 170.18) (end 241.3 175.26) (width 0.25) (layer "F.Cu") (net 25))
@@
   (segment (start 246.38 175.26) (end 243.84 175.26) (width 0.25) (layer "F.Cu") (net 25))
   (segment (start 248.92 170.18) (end 243.84 175.26) (width 0.25) (layer "F.Cu") (net 25))
+  (segment (start 254 187.96) (end 254 182.88) (width 0.25) (layer "F.Cu") (net 25))
+  (segment (start 254 182.88) (end 246.38 175.26) (width 0.25) (layer "F.Cu") (net 25))
   (segment (start 248.92 167.64) (end 248.92 170.18) (width 0.25) (layer "F.Cu") (net 25))
   (segment (start 226.06 175.26) (end 220.98 170.18) (width 0.25) (layer "F.Cu") (net 25))
@@
   (segment (start 255.415 163.975) (end 248.92 157.48) (width 0.25) (layer "B.Cu") (net 26))
   (segment (start 248.92 165.1) (end 248.92 157.48) (width 0.25) (layer "B.Cu") (net 26))
+  (segment (start 243.84 185.42) (end 246.38 187.96) (width 0.25) (layer "F.Cu") (net 27))
+  (segment (start 238.76 185.42) (end 243.84 185.42) (width 0.25) (layer "F.Cu") (net 27))
   (segment (start 237.345 171.305) (end 237.345 168.765) (width 0.25) (layer "B.Cu") (net 27))
-  (segment (start 254 187.96) (end 237.345 171.305) (width 0.25) (layer "B.Cu") (net 27))
+  (segment (start 246.38 180.34) (end 246.38 187.96) (width 0.25) (layer "B.Cu") (net 27))
   (segment (start 237.345 168.765) (end 235.754009 168.765) (width 0.25) (layer "B.Cu") (net 27))
   (segment (start 235.095 166.515) (end 220.98 152.4) (width 0.25) (layer "B.Cu") (net 27))
+  (segment (start 237.345 171.305) (end 246.38 180.34) (width 0.25) (layer "B.Cu") (net 27))
   (segment (start 235.095 168.105991) (end 235.095 166.515) (width 0.25) (layer "B.Cu") (net 27))
   (segment (start 235.754009 168.765) (end 235.095 168.105991) (width 0.25) (layer "B.Cu") (net 27))
@@
   (segment (start 221.06 185.42) (end 221.06 172.8) (width 0.25) (layer "F.Cu") (net 30))
   (segment (start 221.06 172.8) (end 220.98 172.72) (width 0.25) (layer "F.Cu") (net 30))
-  (segment (start 243.84 185.42) (end 246.38 187.96) (width 0.25) (layer "F.Cu") (net 31))
-  (segment (start 238.76 185.42) (end 243.84 185.42) (width 0.25) (layer "F.Cu") (net 31))
   (zone (net 25) (net_name "GND") (layer "B.Cu") (hatch edge 0.5)
     (connect_pads (clearance 0.5))
