File: SYS_DEV/Columbia/V0/V0.6/V0.6.3/sensors/hardware/PCB/smart penetrometer/smart penetrometer.kicad_pro/smart penetrometer.kicad_pro.kicad_pcb (KiCad board)
At the start: 4 copper layers, 29 x 93.3 mm, 36 parts, among them J1 RTD, J2 Conn_01x02, J3 Conn_01x02, J4 GEO, J5 Conn_02x04, J6 EC, U1 LM321, U2 ADP124ARHZ-3.3-R7, U3 SN74LVC8T245DGVR, U4 DS3231M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

Commit message: pcb update
Routing:
- net GND: track 39.2 -> 36.7 mm, vias 37 -> 38
- net NCLK: track 13.0 -> 14.9 mm
Changed lines of the file:
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@@
+	)
+	(segment
+		(start 174.4218 127.9398)
+		(end 174.498 128.016)
+		(width 0.2)
+		(layer "F.Cu")
+		(net 4)
+	)
+	(segment
+		(start 175.492001 126.259999)
+		(end 175.514 126.238)
+		(width 0.2)
+		(layer "F.Cu")
+		(net 4)
+	)
+	(segment
+		(start 174.4218 126.492)
+		(end 174.4218 126.660001)
+		(width 0.2)
+		(layer "F.Cu")
+		(net 4)
 	)
 	(segment
@@
 	)
 	(segment
-		(start 174.4218 126.259999)
-		(end 176.043999 126.259999)
-		(width 0.2)
-		(layer "F.Cu")
-		(net 4)
-	)
-	(segment
 		(start 187.61 82.781)
 		(end 189.461 82.781)
@@
 	(segment
 		(start 174.4218 126.259999)
-		(end 174.4218 126.660001)
-		(width 0.2)
-		(layer "F.Cu")
-		(net 4)
-	)
-	(segment
-		(start 176.043999 126.259999)
-		(end 178.562 128.778)
+		(end 175.492001 126.259999)
+		(width 0.2)
+		(layer "F.Cu")
+		(net 4)
+	)
+	(segment
+		(start 174.4218 126.492)
+		(end 174.4218 127.9398)
+		(width 0.2)
+		(layer "F.Cu")
+		(net 4)
+	)
+	(segment
+		(start 174.4218 126.259999)
+		(end 174.4218 126.492)
 		(width 0.2)
 		(layer "F.Cu")
@@
 	)
 	(via
+		(at 175.514 126.238)
+		(size 0.8)
+		(drill 0.4)
+		(layers "F.Cu" "B.Cu")
+		(free yes)
+		(net 4)
+	)
+	(via
 		(at 166.8 108.78)
 		(size 0.8)
@@
 	)
 	(segment
-		(start 175.768 124.206)
-		(end 179.578 128.016)
+		(start 179.1291 128.778)
+		(end 183.896 128.778)
 		(width 0.2)
 		(layer "F.Cu")
@@
 	)
 	(segment
-		(start 175.13 123.06)
-		(end 175.768 123.698)
+		(start 176.022 125.6709)
+		(end 179.1291 128.778)
 		(width 0.2)
 		(layer "F.Cu")
@@
 	)
 	(segment
-		(start 175.768 123.698)
-		(end 175.768 124.206)
+		(start 183.896 128.778)
+		(end 184.685 127.989)
 		(width 0.2)
 		(layer "F.Cu")
@@
 	)
 	(segment
-		(start 183.764 128.016)
+		(start 184.685 127.989)
 		(end 184.685 127.095)
 		(width 0.2)
@@
 	)
 	(segment
-		(start 179.578 128.016)
-		(end 183.764 128.016)
-		(width 0.2)
-		(layer "F.Cu")
+		(start 176.022 123.952)
+		(end 176.022 125.6709)
+		(width 0.2)
+		(layer "F.Cu")
+		(net 50)
+	)
+	(segment
+		(start 175.13 123.06)
+		(end 176.022 123.952)
+		(width 0.2)
+		(layer "F.Cu")
