File: SYS_DEV/Columbia/V0/V0.6/V0.6.3/sensors/hardware/PCB/smart penetrometer/smart penetrometer.kicad_pro/smart penetrometer.kicad_pro.kicad_sch (KiCad schematic)
At the start: 34 parts, among them J1 RTD, J2 Conn_01x02, J3 Conn_01x02, J4 GEO, J5 Conn_02x04, J6 EC, U1 LM321, U2 ADP124ARHZ-3.3-R7, U3 SN74LVC8T245DGVR, U4 DS3231M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

Commit message: software update
Connections:
- net NCSN: now also A1.13 (D10); no longer A1.10 (D7)
- net NSD_CS: now also A1.7 (D4); no longer A1.13 (D10)
- no-connect marks 26 -> 27
Changed lines of the file:
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@@
 	)
 	(no_connect
-		(at 165.1 109.22)
+		(at 165.1 116.84)
 	)
 	(no_connect
@@
 	(no_connect
 		(at 101.6 67.818)
+	)
+	(no_connect
+		(at 175.26 88.9)
 	)
 	(no_connect
@@
 	(global_label "NCSN"
 		(shape output)
-		(at 165.1 116.84 180)
-		(fields_autoplaced yes)
-		(effects
-			(font
-				(size 1.27 1.27)
-			)
-			(justify right)
-		)
-		(property "Intersheetrefs" "${INTERSHEET_REFS}"
-			(at 156.9743 116.84 0)
+		(at 165.1 124.46 180)
+		(fields_autoplaced yes)
+		(effects
+			(font
+				(size 1.27 1.27)
+			)
+			(justify right)
+		)
+		(property "Intersheetrefs" "${INTERSHEET_REFS}"
+			(at 156.9743 124.46 0)
 			(effects
 				(font
@@
 	(global_label "NSD_CS"
 		(shape output)
-		(at 165.1 124.46 180)
-		(fields_autoplaced yes)
-		(effects
-			(font
-				(size 1.27 1.27)
-			)
-			(justify right)
-		)
-		(property "Intersheetrefs" "${INTERSHEET_REFS}"
-			(at 154.8577 124.46 0)
-			(effects
-				(font
+		(at 165.1 109.22 180)
+		(fields_autoplaced yes)
+		(effects
+			(font
+				(size 1.27 1.27)
+			)
+			(justify right)
+		)
+		(property "Intersheetrefs" "${INTERSHEET_REFS}"
+			(at 154.8577 109.22 0)
+			(effects
+				(font
